Commit message: created xacro files and filled in rover.urdf.xacro with includes

File: rover_ros2/rover_description/urdf/rover.urdf.xacro (robot description, xacro)
@@ -1,130 +1,8 @@
-<!-- PLEASE NOTE THAT THIS IS JUST COBBLED TOGETHER, I NEED THE ACTUAL URDF FROM JOSE SOMETIME -->
-<robot xmlns:xacro="http://ros.org/wiki/xacro" name="my_rover">
-  <!-- Base link -->
-  <link name="base_link">
-    <visual>
-      <geometry>
-        <box size="0.4 0.3 0.1"/>
-      </geometry>
-      <material name="gray">
-        <color rgba="0.5 0.5 0.5 1.0"/>
-      </material>
-    </visual>
-  </link>
-  <!-- Example wheel -->
-  <link name="front_left_wheel">
-   <visual>
-    <origin rpy="1.5708 0 0" xyz="0 0 0"/>
-    <geometry>
-      <cylinder length="0.05" radius="0.05"/>
-    </geometry>
-    <material name="black">
-      <color rgba="0.1 0.1 0.1 1.0"/>
-    </material>
-  </visual>
-  </link>
-  <joint name="front_left_wheel_joint" type="continuous">
-    <parent link="base_link"/>
-    <child link="front_left_wheel"/>
-    <origin xyz="0.2 0.2 -0.05" rpy="0 0 0"/>
-    <axis xyz="0 1 0"/>
-  </joint>
-  <!-- Repeat for other wheels -->
-  <link name="front_right_wheel">
-   <visual>
-    <origin rpy="1.5708 0 0" xyz="0 0 0"/>
-    <geometry>
-      <cylinder length="0.05" radius="0.05"/>
-    </geometry>
-    <material name="black">
-      <color rgba="0.1 0.1 0.1 1.0"/>
-    </material>
-  </visual>
-  </link>
-  <joint name="front_right_wheel_joint" type="continuous">
-    <parent link="base_link"/>
-    <child link="front_right_wheel"/>
-    <origin xyz="0.2 -0.2 -0.05" rpy="0 0 0"/>
-    <axis xyz="0 1 0"/>
-  </joint>
-  <link name="back_left_wheel">
-   <visual>
-    <origin rpy="1.5708 0 0" xyz="0 0 0"/>
-    <geometry>
-      <cylinder length="0.05" radius="0.05"/>
-    </geometry>
-    <material name="black">
-      <color rgba="0.1 0.1 0.1 1.0"/>
-    </material>
-  </visual>
-  </link>
-  <joint name="back_left_wheel_joint" type="continuous">
-    <parent link="base_link"/>
-    <child link="back_left_wheel"/>
-    <origin xyz="-0.2 0.2 -0.05" rpy="0 0 0"/>
-    <axis xyz="0 1 0"/>
-  </joint>
-  <link name="back_right_wheel">
-   <visual>
-    <origin rpy="1.5708 0 0" xyz="0 0 0"/>
-    <geometry>
-      <cylinder length="0.05" radius="0.05"/>
-    </geometry>
-    <material name="black">
-      <color rgba="0.1 0.1 0.1 1.0"/>
-    </material>
-  </visual>
-  </link>
-  <joint name="back_right_wheel_joint" type="continuous">
-    <parent link="base_link"/>
-    <child link="back_right_wheel"/>
-    <origin xyz="-0.2 -0.2 -0.05" rpy="0 0 0"/>
-    <axis xyz="0 1 0"/>
-  </joint>
-  <!-- ros2_control block here -->
-  <ros2_control name="RERASSOR_diff_drive" type="system">
-    <hardware>
-      <plugin>rover_control/RERASSORHardwareInterface</plugin>
-      <param name="front_left_wheel_name">front_left_wheel_joint</param>
-      <param name="front_right_wheel_name">front_right_wheel_joint</param>
-      <param name="back_left_wheel_name">back_left_wheel_joint</param>
-      <param name="back_right_wheel_name">back_right_wheel_joint</param>
-      <param name="device">/dev/ttyACM0</param>
-      <param name="baud_rate">115200</param>
-      <param name="enc_counts_per_rev">2048</param>
-    </hardware>
-    <!-- Joint interface declarations -->
-    <joint name="front_left_wheel_joint">
-      <command_interface name="velocity">
-        <param name="min">-10.0</param>
-        <param name="max">10.0</param>
-      </command_interface>
-      <state_interface name="velocity"/>
-      <state_interface name="position"/>
-    </joint>
-    <joint name="front_right_wheel_joint">
-      <command_interface name="velocity">
-        <param name="min">-10.0</param>
-        <param name="max">10.0</param>
-      </command_interface>
-      <state_interface name="velocity"/>
-      <state_interface name="position"/>
-    </joint>
-    <joint name="back_left_wheel_joint">
-      <command_interface name="velocity">
-        <param name="min">-10.0</param>
-        <param name="max">10.0</param>
-      </command_interface>
-      <state_interface name="velocity"/>
-      <state_interface name="position"/>
-    </joint>
-    <joint name="back_right_wheel_joint">
-      <command_interface name="velocity">
-        <param name="min">-10.0</param>
-        <param name="max">10.0</param>
-      </command_interface>
-      <state_interface name="velocity"/>
-      <state_interface name="position"/>
-    </joint>
-  </ros2_control>
+<?xml version="1.0"?>
+<robot xmlns:xacro="http://ros.org/wiki/xacro" name="re-rassor">
+  <xacro:include filename="rover_core.xacro"/>
+  <xacro:include filename="camera.xacro"/>
+  <xacro:include filename="ros2_control.xacro"/>
+  <!-- Templates -->
+  <xacro:include filename="inertial_macros.xacro"/>
 </robot>

Commit message: fixed issue with chassis_origin parsing

File: rover_ros2/rover_description/urdf/rover.urdf.xacro (robot description, xacro)
@@ -1,8 +1,9 @@
 <?xml version="1.0"?>
 <robot xmlns:xacro="http://ros.org/wiki/xacro" name="re-rassor">
+  <!-- Templates -->
+  <xacro:include filename="inertial_macros.xacro"/>
+  <!-- Parts -->
   <xacro:include filename="rover_core.xacro"/>
   <xacro:include filename="camera.xacro"/>
   <xacro:include filename="ros2_control.xacro"/>
-  <!-- Templates -->
-  <xacro:include filename="inertial_macros.xacro"/>
 </robot>

File: rover_ros2/rover_description/urdf/rover_core.xacro (robot description, xacro)
@@ -22,5 +22,5 @@
     <xacro:property name="chassis_height" value="0.11"/>
     <xacro:property name="chassis_mass" value="0.1"/>
-    <xacro:property name="chassis_origin" value="${chassis_origin}"/>
+    <xacro:property name="chassis_origin" value="0.15 0 0.075"/>
     <xacro:property name="fr_wheel_origin" value="0 0 0"/>
     <xacro:property name="fl_wheel_origin" value="0 0 0"/>
