Commit message: took some basic geometry measurements of parts and started on chassis

File: rover_ros2/rover_description/urdf/rover_core.xacro (robot description, xacro)
@@ -16,5 +16,11 @@
     <!-- BASE -->
     <link name="base_link"/>
-    <!-- CHASSIS (including wheel tubes) -->
+    <!-- CHASSIS -->
+    <joint name="chassis_joint" type="fixed">
+        <parent link="base_link"/>
+        <child link="chassis_link"/>
+        <origin xyz="0 0 0"/>
+    </joint>
+    <!-- WHEEL TUBES -->
     <!-- WHEELS -->
 </robot>

Commit message: added more properties and finished chassis

File: rover_ros2/rover_description/urdf/rover_core.xacro (robot description, xacro)
@@ -12,6 +12,23 @@
     </material>
     <!-- PROPERTIES -->
-    <xacro:property name="wheel_radius" value=""/>
-    <xacro:property name="wheel_length" value=""/>
+    <xacro:property name="wheel_length" value="0.098"/>
+    <xacro:property name="wheel_radius" value="0.115"/>
+    <xacro:property name="wheel_mass" value="0.1"/>
+    <xacro:property name="tube_length" value="0.1"/>
+    <xacro:property name="tube_radius" value="0.065"/>
+    <xacro:property name="tube_mass" value="0.1"/>
+    <xacro:property name="chassis_width" value="0.19"/>
+    <xacro:property name="chassis_length" value="0.37"/>
+    <xacro:property name="chassis_height" value="0.11"/>
+    <xacro:property name="chassis_mass" value="0.1"/>
+    <xacro:property name="chassis_origin" value="${chassis_origin}"/>
+    <xacro:property name="fr_wheel_origin" value="0 0 0"/>
+    <xacro:property name="fl_wheel_origin" value="0 0 0"/>
+    <xacro:property name="br_wheel_origin" value="0 0 0"/>
+    <xacro:property name="bl_wheel_origin" value="0 0 0"/>
+    <xacro:property name="fr_tube_origin" value="0 0 0"/>
+    <xacro:property name="fl_tube_origin" value="0 0 0"/>
+    <xacro:property name="br_tube_origin" value="0 0 0"/>
+    <xacro:property name="bl_tube_origin" value="0 0 0"/>
     <!-- BASE -->
     <link name="base_link"/>
@@ -22,4 +39,25 @@
         <origin xyz="0 0 0"/>
     </joint>
+    <link name="chassis_link">
+        <visual>
+            <origin xyz="${chassis_origin}" rpy="0 0 0"/>
+            <geometry>
+                <box size="${chassis_width} ${chassis_length} ${chassis_height}"/>
+            </geometry>
+            <material name="gray"/>
+        </visual>
+        <collision>
+            <origin xyz="${chassis_origin}" rpy="0 0 0"/>
+            <geometry>
+                <box size="${chassis_width} ${chassis_length} ${chassis_height}"/>
+            </geometry>
+        </collision>
+        <xacro:inertial_box mass="${chassis_mass}" x="${chassis_width}" y="${chassis_length}" z="${chassis_height}">
+            <origin xyz="${chassis_origin}" rpy="0 0 0"/>
+        </xacro:inertial_box>
+    </link>
+    <gazebo reference="chassis_link">
+        <material>Gazebo/Gray</material>
+    </gazebo>
     <!-- WHEEL TUBES -->
     <!-- WHEELS -->

Commit message: removed properties and materials from rover_core

File: rover_ros2/rover_description/urdf/rover_core.xacro (robot description, xacro)
@@ -1,34 +1,4 @@
 <?xml version="1.0"?>
 <robot xmlns:xacro="http://www.ros.org/wiki/xacro">
-    <!-- MATERIALS -->
-    <material name="gray">
-        <color rgba="${192/255} ${192/255} ${192/255} 1.0"/>
-    </material>
-    <material name="slate_gray">
-        <color rgba="${112/255} ${128/255} ${144/255} 1.0"/>
-    </material>
-    <material name="black">
-        <color rgba="0.0 0.0 0.0 1.0"/>
-    </material>
-    <!-- PROPERTIES -->
-    <xacro:property name="wheel_length" value="0.098"/>
-    <xacro:property name="wheel_radius" value="0.115"/>
-    <xacro:property name="wheel_mass" value="0.1"/>
-    <xacro:property name="tube_length" value="0.1"/>
-    <xacro:property name="tube_radius" value="0.065"/>
-    <xacro:property name="tube_mass" value="0.1"/>
-    <xacro:property name="chassis_width" value="0.19"/>
-    <xacro:property name="chassis_length" value="0.37"/>
-    <xacro:property name="chassis_height" value="0.11"/>
-    <xacro:property name="chassis_mass" value="0.1"/>
-    <xacro:property name="chassis_origin" value="0.15 0 0.075"/>
-    <xacro:property name="fr_wheel_origin" value="0 0 0"/>
-    <xacro:property name="fl_wheel_origin" value="0 0 0"/>
-    <xacro:property name="br_wheel_origin" value="0 0 0"/>
-    <xacro:property name="bl_wheel_origin" value="0 0 0"/>
-    <xacro:property name="fr_tube_origin" value="0 0 0"/>
-    <xacro:property name="fl_tube_origin" value="0 0 0"/>
-    <xacro:property name="br_tube_origin" value="0 0 0"/>
-    <xacro:property name="bl_tube_origin" value="0 0 0"/>
     <!-- BASE -->
     <link name="base_link"/>
