Commit message: finished modeling the tubes

File: rover_ros2/rover_description/urdf/config.xacro (robot description, xacro)
@@ -19,18 +19,18 @@
     <xacro:property name="wheel_mass" value="0.1"/>
     <xacro:property name="tube_length" value="0.1"/>
-    <xacro:property name="tube_radius" value="0.065"/>
+    <xacro:property name="tube_radius" value="0.0325"/>
     <xacro:property name="tube_mass" value="0.1"/>
-    <xacro:property name="chassis_width" value="0.19"/>
-    <xacro:property name="chassis_length" value="0.37"/>
+    <xacro:property name="chassis_width" value="0.37"/>
+    <xacro:property name="chassis_length" value="0.19"/>
     <xacro:property name="chassis_height" value="0.11"/>
     <xacro:property name="chassis_mass" value="0.1"/>
-    <xacro:property name="chassis_origin" value="0.15 0 0.075"/>
+    <xacro:property name="chassis_origin" value="0 0 0.055"/>
     <xacro:property name="fr_wheel_origin" value="0 0 0"/>
     <xacro:property name="fl_wheel_origin" value="0 0 0"/>
     <xacro:property name="br_wheel_origin" value="0 0 0"/>
     <xacro:property name="bl_wheel_origin" value="0 0 0"/>
-    <xacro:property name="fr_tube_origin" value="0 0 0"/>
-    <xacro:property name="fl_tube_origin" value="0 0 0"/>
-    <xacro:property name="br_tube_origin" value="0 0 0"/>
-    <xacro:property name="bl_tube_origin" value="0 0 0"/>
+    <xacro:property name="fr_tube_origin" value="0.15 -0.145 ${tube_radius}"/>
+    <xacro:property name="fl_tube_origin" value="0.15 0.145 ${tube_radius}"/>
+    <xacro:property name="br_tube_origin" value="-0.15 -0.145 ${tube_radius}"/>
+    <xacro:property name="bl_tube_origin" value="-0.15 0.145 ${tube_radius}"/>
 </robot>

File: rover_ros2/rover_description/urdf/cylinder_macro.xacro (robot description, xacro)
@@ -1,5 +1,5 @@
 <?xml version="1.0"?>
 <robot xmlns:xacro="http://www.ros.org/wiki/xacro">
-    <xacro:macro name="wheel" params="mass radius length material *origin">
+    <xacro:macro name="cylinder_macro" params="mass radius length material *origin">
         <visual>
             <geometry>

File: rover_ros2/rover_description/urdf/rover.urdf.xacro (robot description, xacro)
@@ -5,4 +5,5 @@
   <!-- Templates -->
   <xacro:include filename="inertial_macros.xacro"/>
+  <xacro:include filename="cylinder_macro.xacro"/>
   <!-- Parts -->
   <xacro:include filename="rover_core.xacro"/>

File: rover_ros2/rover_description/urdf/rover_core.xacro (robot description, xacro)
@@ -24,5 +24,5 @@
         </collision>
         <xacro:inertial_box mass="${chassis_mass}" x="${chassis_width}" y="${chassis_length}" z="${chassis_height}">
-            <origin xyz="${chassis_origin}" rpy="0 0 0"/>
+            <origin xyz="0 0 0" rpy="0 0 0"/>
         </xacro:inertial_box>
     </link>
@@ -31,4 +31,52 @@
     </gazebo>
     <!-- WHEEL TUBES -->
+    <joint name="fr_tube_joint" type="fixed">
+        <parent link="chassis_link"/>
+        <child link="fr_tube_link"/>
+        <origin xyz="${fr_tube_origin}" rpy="${pi/2} 0 0"/>
+    </joint>
+    <link name="fr_tube_link">
+        <xacro:cylinder_macro
+            mass="${tube_mass}" radius="${tube_radius}"
+            length="${tube_length}" material="slate_gray">
+            <origin xyz="0 0 0" rpy="0 0 0"/>
+        </xacro:cylinder_macro>
+    </link>
+    <joint name="fl_tube_joint" type="fixed">
+        <parent link="chassis_link"/>
+        <child link="fl_tube_link"/>
+        <origin xyz="${fl_tube_origin}" rpy="${pi/2} 0 0"/>
+    </joint>
+    <link name="fl_tube_link">
+        <xacro:cylinder_macro
+            mass="${tube_mass}" radius="${tube_radius}"
+            length="${tube_length}" material="slate_gray">
+            <origin xyz="0 0 0" rpy="0 0 0"/>
+        </xacro:cylinder_macro>
+    </link>
+    <joint name="br_tube_joint" type="fixed">
+        <parent link="chassis_link"/>
+        <child link="br_tube_link"/>
+        <origin xyz="${br_tube_origin}" rpy="${pi/2} 0 0"/>
+    </joint>
+    <link name="br_tube_link">
+        <xacro:cylinder_macro
+            mass="${tube_mass}" radius="${tube_radius}"
+            length="${tube_length}" material="slate_gray">
+            <origin xyz="0 0 0" rpy="0 0 0"/>
+        </xacro:cylinder_macro>
+    </link>
+    <joint name="bl_tube_joint" type="fixed">
+        <parent link="chassis_link"/>
+        <child link="bl_tube_link"/>
+        <origin xyz="${bl_tube_origin}" rpy="${pi/2} 0 0"/>
+    </joint>
+    <link name="bl_tube_link">
+        <xacro:cylinder_macro
+            mass="${tube_mass}" radius="${tube_radius}"
+            length="${tube_length}" material="slate_gray">
+            <origin xyz="0 0 0" rpy="0 0 0"/>
+        </xacro:cylinder_macro>
+    </link>
     <!-- WHEELS -->
 </robot>

Commit message: made the rsp launch file

File: rover_ros2/rover_description/urdf/config.xacro (robot description, xacro)
@@ -26,5 +26,5 @@
     <xacro:property name="chassis_mass" value="0.1"/>
     <xacro:property name="chassis_origin" value="0 0 0.055"/>
-    <xacro:property name="fr_wheel_origin" value="0 0 0"/>
+    <xacro:property name="fr_wheel_origin" value="0 ${tube_length/2} 0"/>
     <xacro:property name="fl_wheel_origin" value="0 0 0"/>
     <xacro:property name="br_wheel_origin" value="0 0 0"/>

File: rover_ros2/rover_description/urdf/rover_core.xacro (robot description, xacro)
@@ -80,3 +80,17 @@
     </link>
     <!-- WHEELS -->
+    <joint name="fr_wheel_joint" type="continuous">
+        <parent link="fr_tube_link"/>
+        <child link="fr_wheel_link"/>
+        <origin xyz="${fr_wheel_origin}" rpy="0 0 0"/>
+        <axis xyz="0 0 1"/>
+        <limit effort="5" velocity="20"/>
+    </joint>
+    <link name="fr_wheel_link">
+        <xacro:cylinder_macro
+            mass="${wheel_mass}" radius="${wheel_radius}"
+            length="${wheel_length}" material="gray">
+            <origin xyz="0 0 0" rpy="0 0 0"/>
+        </xacro:cylinder_macro>
+    </link>
 </robot>
