Commit message: updated the rerassor urdf to remove meshes

File: rover_ros2/rover_description/urdf/materials.xacro (robot description, xacro)
@@ -26,3 +26,9 @@
         <color rgba="1.0 1.0 1.0 1.0"/>
     </material>
+    <material name="chassis_color">
+        <color rgba="0.6 0.6 0.6 1.0"/>  <!-- gray -->
+    </material>
+    <material name="wheel_color">
+        <color rgba="0.0 0.0 0.0 1.0"/>  <!-- black -->
+    </material>
 </robot>

File: rover_ros2/rover_description/urdf/rerassor.urdf.xacro (robot description, xacro)
@@ -52,5 +52,5 @@
 			<origin xyz="0 0 0" rpy=" 0 0 0"/>
 			<geometry>
-       			<mesh filename="file://meshes/base_unit.dae" scale="0.01 0.01 0.01"></mesh>
+				<box size="0.4 0.3 0.2"/>
 			</geometry>
 		</collision>
@@ -58,6 +58,7 @@
 			<origin xyz="0 0 0" rpy=" 0 0 0"/>
 			<geometry>
-        		<mesh filename="file://meshes/base_unit.dae" scale="0.01 0.01 0.01"></mesh>
-			</geometry>
+				<box size="0.4 0.3 0.2"/>
+			</geometry>
+			<material name="chassis_color"/>
 		</visual>
 	</link>
@@ -79,11 +80,12 @@
 			<origin xyz="0 0 0" rpy="0 0 0"/>
 			<geometry>
-				<mesh filename="file://meshes/wheel.dae" scale="0.01 0.01 0.01"/>
-			</geometry>
-		</visual>
-		<collision name="collision">
-			<origin xyz="0 0 0" rpy="0 0 0"/>
-			<geometry>
-				<mesh filename="file://meshes/wheel.dae" scale="0.01 0.01 0.01"/>
+				<cylinder radius="0.1" length="0.05"/>  <!-- Wheel approx: 20cm diameter, 5cm thick -->
+			</geometry>
+			<material name="wheel_color"/>
+		</visual>
+		<collision name="collision">
+			<origin xyz="0 0 0" rpy="0 0 0"/>
+			<geometry>
+				<cylinder radius="0.1" length="0.05"/>
 			</geometry>
 			<surface>
@@ -119,11 +121,12 @@
 			<origin xyz="0 0 0" rpy="0 0 0"/>
 			<geometry>
-				<mesh filename="file://meshes/wheel.dae" scale="0.01 0.01 0.01"/>
-			</geometry>
-		</visual>
-		<collision name="collision">
-			<origin xyz="0 0 0" rpy="0 0 0"/>
-			<geometry>
-				<mesh filename="file://meshes/wheel.dae" scale="0.01 0.01 0.01"/>
+				<cylinder radius="0.1" length="0.05"/>
+			</geometry>
+			<material name="wheel_color"/>
+		</visual>
+		<collision name="collision">
+			<origin xyz="0 0 0" rpy="0 0 0"/>
+			<geometry>
+				<cylinder radius="0.1" length="0.05"/>
 			</geometry>
 			<surface>
@@ -159,11 +162,12 @@
 			<origin xyz="0 0 0" rpy="0 0 0"/>
 			<geometry>
-				<mesh filename="file://meshes/wheel.dae" scale="0.01 0.01 0.01"/>
-			</geometry>
-		</visual>
-		<collision name="collision">
-			<origin xyz="0 0 0" rpy="0 0 0"/>
-			<geometry>
-				<mesh filename="file://meshes/wheel.dae" scale="0.01 0.01 0.01"/>
+				<cylinder radius="0.1" length="0.05"/>
+			</geometry>
+			<material name="wheel_color"/>
+		</visual>
+		<collision name="collision">
+			<origin xyz="0 0 0" rpy="0 0 0"/>
+			<geometry>
+				<cylinder radius="0.1" length="0.05"/>
 			</geometry>
 			<surface>
@@ -199,11 +203,12 @@
 			<origin xyz="0 0 0" rpy="0 0 0"/>
 			<geometry>
-				<mesh filename="file://meshes/wheel.dae" scale="0.01 0.01 0.01"/>
-			</geometry>
-		</visual>
-		<collision name="collision">
-			<origin xyz="0 0 0" rpy="0 0 0"/>
-			<geometry>
-				<mesh filename="file://meshes/wheel.dae" scale="0.01 0.01 0.01"/>
+				<cylinder radius="0.1" length="0.05"/>
+			</geometry>
+			<material name="wheel_color"/>
+		</visual>
+		<collision name="collision">
+			<origin xyz="0 0 0" rpy="0 0 0"/>
+			<geometry>
+				<cylinder radius="0.1" length="0.05"/>
 			</geometry>
 			<surface>

Commit message: Revert "updated the rerassor urdf to remove meshes"
This reverts commit be9e5e833e6e37bc2f9bf4ce21fd192e0a5b240a.

File: rover_ros2/rover_description/urdf/materials.xacro (robot description, xacro)
@@ -26,9 +26,3 @@
         <color rgba="1.0 1.0 1.0 1.0"/>
     </material>
-    <material name="chassis_color">
-        <color rgba="0.6 0.6 0.6 1.0"/>  <!-- gray -->
-    </material>
-    <material name="wheel_color">
-        <color rgba="0.0 0.0 0.0 1.0"/>  <!-- black -->
-    </material>
 </robot>

File: rover_ros2/rover_description/urdf/rerassor.urdf.xacro (robot description, xacro)
@@ -52,5 +52,5 @@
 			<origin xyz="0 0 0" rpy=" 0 0 0"/>
 			<geometry>
-				<box size="0.4 0.3 0.2"/>
+       			<mesh filename="file://meshes/base_unit.dae" scale="0.01 0.01 0.01"></mesh>
 			</geometry>
 		</collision>
@@ -58,7 +58,6 @@
 			<origin xyz="0 0 0" rpy=" 0 0 0"/>
 			<geometry>
-				<box size="0.4 0.3 0.2"/>
-			</geometry>
-			<material name="chassis_color"/>
+        		<mesh filename="file://meshes/base_unit.dae" scale="0.01 0.01 0.01"></mesh>
+			</geometry>
 		</visual>
 	</link>
@@ -80,12 +79,11 @@
 			<origin xyz="0 0 0" rpy="0 0 0"/>
 			<geometry>
-				<cylinder radius="0.1" length="0.05"/>  <!-- Wheel approx: 20cm diameter, 5cm thick -->
-			</geometry>
-			<material name="wheel_color"/>
-		</visual>
-		<collision name="collision">
-			<origin xyz="0 0 0" rpy="0 0 0"/>
-			<geometry>
-				<cylinder radius="0.1" length="0.05"/>
+				<mesh filename="file://meshes/wheel.dae" scale="0.01 0.01 0.01"/>
+			</geometry>
+		</visual>
+		<collision name="collision">
+			<origin xyz="0 0 0" rpy="0 0 0"/>
+			<geometry>
+				<mesh filename="file://meshes/wheel.dae" scale="0.01 0.01 0.01"/>
 			</geometry>
 			<surface>
@@ -121,12 +119,11 @@
 			<origin xyz="0 0 0" rpy="0 0 0"/>
 			<geometry>
-				<cylinder radius="0.1" length="0.05"/>
-			</geometry>
-			<material name="wheel_color"/>
-		</visual>
-		<collision name="collision">
-			<origin xyz="0 0 0" rpy="0 0 0"/>
-			<geometry>
-				<cylinder radius="0.1" length="0.05"/>
+				<mesh filename="file://meshes/wheel.dae" scale="0.01 0.01 0.01"/>
+			</geometry>
+		</visual>
+		<collision name="collision">
+			<origin xyz="0 0 0" rpy="0 0 0"/>
+			<geometry>
+				<mesh filename="file://meshes/wheel.dae" scale="0.01 0.01 0.01"/>
 			</geometry>
 			<surface>
@@ -162,12 +159,11 @@
 			<origin xyz="0 0 0" rpy="0 0 0"/>
 			<geometry>
-				<cylinder radius="0.1" length="0.05"/>
-			</geometry>
-			<material name="wheel_color"/>
-		</visual>
-		<collision name="collision">
-			<origin xyz="0 0 0" rpy="0 0 0"/>
-			<geometry>
-				<cylinder radius="0.1" length="0.05"/>
+				<mesh filename="file://meshes/wheel.dae" scale="0.01 0.01 0.01"/>
+			</geometry>
+		</visual>
+		<collision name="collision">
+			<origin xyz="0 0 0" rpy="0 0 0"/>
+			<geometry>
+				<mesh filename="file://meshes/wheel.dae" scale="0.01 0.01 0.01"/>
 			</geometry>
 			<surface>
@@ -203,12 +199,11 @@
 			<origin xyz="0 0 0" rpy="0 0 0"/>
 			<geometry>
-				<cylinder radius="0.1" length="0.05"/>
-			</geometry>
-			<material name="wheel_color"/>
-		</visual>
-		<collision name="collision">
-			<origin xyz="0 0 0" rpy="0 0 0"/>
-			<geometry>
-				<cylinder radius="0.1" length="0.05"/>
+				<mesh filename="file://meshes/wheel.dae" scale="0.01 0.01 0.01"/>
+			</geometry>
+		</visual>
+		<collision name="collision">
+			<origin xyz="0 0 0" rpy="0 0 0"/>
+			<geometry>
+				<mesh filename="file://meshes/wheel.dae" scale="0.01 0.01 0.01"/>
 			</geometry>
 			<surface>
