Commit message: fixed imu having mismatched variables with cameras

File: rover_ros2/rover_description/urdf/imu.xacro (robot description, xacro)
@@ -2,5 +2,5 @@
 <robot name="rerassor" xmlns:xacro="http://www.ros.org/wiki/xacro">
     <!-- Macro to add an IMU sensor to a given parent link -->
-    <xacro:macro name="rerassor_imu" params="imu_prefix parent xyz rpy">
+    <xacro:macro name="rerassor_imu" params="imu_prefix parent imu_size xyz rpy">
         <link name="${imu_prefix}_link">
             <inertial>
@@ -12,5 +12,5 @@
                 <origin xyz="0 0 0" rpy="0 0 0"/>
                 <geometry>
-                    <box size="${camera_size} ${camera_size} ${camera_size}"/>
+                    <box size="${imu_size} ${imu_size} ${imu_size}"/>
                 </geometry>
             </collision>
@@ -18,5 +18,5 @@
                 <origin xyz="0 0 0" rpy="0 0 0"/>
                 <geometry>
-                    <box size="${camera_size} ${camera_size} ${camera_size}"/>
+                    <box size="${imu_size} ${imu_size} ${imu_size}"/>
                 </geometry>
                 <material name="green"/>

File: rover_ros2/rover_description/urdf/rerassor.urdf.xacro (robot description, xacro)
@@ -186,5 +186,5 @@
     <xacro:include filename="$(find rover_description)/urdf/imu.xacro" />
     <xacro:rerassor_imu imu_prefix="imu_link" parent="base_link"
-                        xyz="0 0 0.2" rpy="0 0 0" />
+                        imu_size="${cameraSize}" xyz="0 0 0.2" rpy="0 0 0" />
     <!-- Depth camera sensor (Gazebo Sim format) -->
     <gazebo reference="depth_camera_optical">
