Commit message: it launches but its just a big yellow box with wheels. not what i wanted

File: rover_ros2/rover_description/urdf/macros.xacro (robot description, xacro)
@@ -4,13 +4,17 @@
     <!-- Inertia Tensors Used: https://en.wikipedia.org/wiki/List_of_moments_of_inertia#List_of_3D_inertia_tensors -->
     <xacro:macro name="cylinder_inertia" params="m r h">
+        <mass value="${m}"/>
         <inertia ixx="${m*((3*r*r)+(h*h))/12}" ixy = "0"                 ixz = "0" iyy="${m*((3*r*r)+(h*h))/12}" iyz = "0" izz="${(m*(r*r))/2}" />
     </xacro:macro>
     <xacro:macro name="box_inertia" params="m x y z">
+        <mass value="${m}"/>
         <inertia ixx="${m*(y*y+z*z)/12}" ixy = "0" ixz = "0" iyy="${m*(x*x+z*z)/12}" iyz = "0" izz="${m*(x*x+z*z)/12}" />
     </xacro:macro>
     <xacro:macro name="sphere_inertia" params="m r">
+        <mass value="${m}"/>
         <inertia ixx="${2*m*r*r/5}" ixy = "0" ixz = "0" iyy="${2*m*r*r/5}" iyz = "0" izz="${2*m*r*r/5}" />
     </xacro:macro>
     <xacro:macro name="slender_rod_along_y_inertia" params="m l mass_about">
+        <mass value="${m}"/>
         <xacro:if value="${mass_about == 'end'}">
             <inertia ixx="${1/3*m*(l*l)}" ixy = "0"
