Commit message: fix: correct joint name from 'base_link_fixed' to 'base_link' in URDF

File: rover_ros2/rover_description/urdf/rerassor.urdf.xacro (robot description, xacro)
@@ -43,5 +43,5 @@
     </link>
     <!-- Base link is root of the robot -->
-    <joint name="base_link_fixed" type="fixed">
+    <joint name="base_link" type="fixed">
         <parent link="world"/>
         <child link="base_link"/>

Commit message: changed base_link to chassis_link and added an empty base_link as its parent

File: rover_ros2/rover_description/urdf/rerassor.urdf.xacro (robot description, xacro)
@@ -10,6 +10,7 @@
     <xacro:property name="camera_y" value="0.3"/>
     <xacro:property name="camera_z" value="1.5"/>
+	<link name="base_link"></link>
     <!-- Base link (main body) -->
-    <link name="base_link">
+    <link name="chassis_link">
         <inertial>
             <origin xyz="0 0 0" rpy="0 0 0"/>
@@ -17,5 +18,5 @@
             <xacro:call macro="box_inertia" m="50" x="1.0" y="1.5" z="0.3"/>
         </inertial>
-        <collision name='base_link_collision'>
+        <collision name='chassis_link_collision'>
             <origin xyz="0 0 0" rpy="0 0 0"/>
             <geometry>
@@ -34,5 +35,5 @@
             </surface>
         </collision>
-        <visual name='base_link_visual'>
+        <visual name='chassis_link_visual'>
             <origin xyz="0 0 0" rpy="0 0 0"/>
             <geometry>
@@ -43,9 +44,9 @@
     </link>
     <!-- Base link is root of the robot -->
-    <joint name="base_link" type="fixed">
-        <parent link="world"/>
-        <child link="base_link"/>
-    </joint>
-    <!-- Four Wheels attached to base_link -->
+    <joint name="chassis_joint" type="fixed">
+        <parent link="base_link"/>
+        <child link="chassis_link"/>
+    </joint>
+    <!-- Four Wheels attached to chassis_link -->
     <!-- Left Front Wheel -->
     <link name="left_wheel_front_link">
@@ -181,9 +182,9 @@
     <!-- Depth camera attachment -->
     <xacro:include filename="$(find rover_description)/urdf/camera.xacro" />
-    <xacro:rerassor_camera camera_prefix="depth_camera" parent="base_link"
+    <xacro:rerassor_camera camera_prefix="depth_camera" parent="chassis_link"
                            x="${camera_x}" y="${camera_y}" z="${camera_z}" />
     <!-- IMU attachment -->
     <xacro:include filename="$(find rover_description)/urdf/imu.xacro" />
-    <xacro:rerassor_imu imu_prefix="imu_link" parent="base_link"
+    <xacro:rerassor_imu imu_prefix="imu_link" parent="chassis_link"
                         imu_size="${cameraSize}" xyz="0 0 0.2" rpy="0 0 0" />
     <!-- Depth camera sensor (Gazebo Sim format) -->

Commit message: working on making the simplified urdfs

File: rover_ros2/rover_description/urdf/rerassor.urdf.xacro (robot description, xacro)
@@ -1,13 +1,8 @@
 <?xml version='1.0'?>
 <robot name="rerassor" xmlns:xacro="http://www.ros.org/wiki/xacro">
-    <xacro:property name="cameraSize" value="0.01"/>
-    <xacro:property name="cameraMass" value="0.1"/>
-    <xacro:include filename="$(find rover_description)/urdf/macros.xacro" />
-    <xacro:include filename="$(find rover_description)/urdf/materials.xacro" />
-    <xacro:include filename="$(find rover_description)/urdf/imu.xacro" />
-    <!-- Camera position guesstimated to align with the mast -->
-    <xacro:property name="camera_x" value="0.0"/>
-    <xacro:property name="camera_y" value="0.3"/>
-    <xacro:property name="camera_z" value="1.5"/>
+    <xacro:include filename="$(find rover_description)/urdf/inertial_macros.xacro"/>
+    <xacro:include filename="$(find rover_description)/urdf/properties.xacro"/>
+    <xacro:include filename="$(find rover_description)/urdf/wheel.xacro"/>
+    <xacro:include filename="$(find rover_description)/urdf/wheel_arm.xacro"/>
 	<link name="base_link"></link>
     <!-- Base link (main body) -->
@@ -48,6 +43,12 @@
         <child link="chassis_link"/>
     </joint>
-    <!-- Four Wheels attached to chassis_link -->
-    <!-- Left Front Wheel -->
+    <!-- Wheel arms -->
+    <xacro:wheel_arm arm_name="fl_wheel_arm" parent_link="chassis_link"
+                length="1.0" radius="0.1" mass="5.0"
+                origin_xyz="1.5 1.2 0.0" origin_rpy="0 ${pi/2} 0"/>
+    <!-- Wheels -->
+    <xacro:wheel wheel_name="fl_wheel" parent_link="fl_wheel_arm_link"
+             radius="0.3" width="0.2" mass="5.0"
+             origin_xyz="0 0 ${-0.5}" origin_rpy="0 0 0"/>
     <link name="left_wheel_front_link">
         <inertial>

File: rover_ros2/rover_description/urdf/wheel.xacro (robot description, xacro)
@@ -1,40 +1,29 @@
 <?xml version='1.0'?>
 <robot name="rerassor" xmlns:xacro="http://www.ros.org/wiki/xacro">
-    <!-- Macro defining the wheel geometry (cylinder) -->
-    <xacro:macro name="wheel_mesh">
-        <cylinder radius="0.18" length="0.2"/>
-    </xacro:macro>
-    <!-- The wheel module macro (if it were used) -->
-    <xacro:macro name="rerassor_wheel" params="wheel_prefix parent xyz rpy yaw">
-        <link name="${wheel_prefix}">
+    <!-- wheel.xacro -->
+    <xacro:macro name="wheel" params="wheel_name parent_link radius width mass origin_xyz origin_rpy">
+        <link name="${wheel_name}_link">
             <inertial>
                 <origin xyz="0 0 0" rpy="0 0 0"/>
-                <xacro:call macro="cylinder_inertia" m="5" r="0.18" h="0.2"/>
+                <mass value="${mass}"/>
+                <xacro:cylinder_inertia m="${mass}" r="${radius}" h="${width}"/>
             </inertial>
-            <visual name="${wheel_prefix}_visual">
-                <origin xyz="0 0 0" rpy="0 0 ${yaw}"/>
-                <geometry>
-                    <xacro:wheel_mesh/>
-                </geometry>
+            <visual>
+                <origin xyz="0 0 0" rpy="0 0 0"/>
+                <geometry><cylinder radius="${radius}" length="${width}"/></geometry>
+                <material name="Grey"/>
             </visual>
-            <collision name="${wheel_prefix}_collision">
-                <origin xyz="0 0 0" rpy="0 0 ${yaw}"/>
-                <geometry>
-                    <xacro:wheel_mesh/>
-                </geometry>
-                <surface>
-                    <friction>
-                        <mu>1.5</mu>
-                        <mu2>1.5</mu2>
-                    </friction>
-                </surface>
+            <collision>
+                <origin xyz="0 0 0" rpy="0 0 0"/>
+                <geometry><cylinder radius="${radius}" length="${width}"/></geometry>
+                <surface><friction><mu>1.5</mu><mu2>1.5</mu2></friction></surface>
             </collision>
         </link>
-        <joint name="${wheel_prefix}_joint" type="continuous">
-            <origin xyz="${xyz}" rpy="${rpy}"/>
-            <parent link="${parent}"/>
-            <child link="${wheel_prefix}"/>
-            <axis xyz="0 1 0"/>
-            <limit effort="1000" velocity="5"/>
+        <joint name="${wheel_name}_joint" type="continuous">
+            <parent link="${parent_link}"/>
+            <child link="${wheel_name}_link"/>
+            <origin xyz="${origin_xyz}" rpy="${origin_rpy}"/>
+            <axis xyz="0 1 0"/>  <!-- assuming wheel rotates about the Y-axis of arm frame -->
+            <dynamics damping="0.2"/>
         </joint>
     </xacro:macro>
