Commit message: updated xacros to not use meshes and use gazebo harmonic

File: rover_ros2/rover_description/urdf/camera.xacro (robot description, xacro)
@@ -1,13 +1,13 @@
 <?xml version='1.0'?>
-<robot name="rerassor"
-    xmlns:xacro="http://www.ros.org/wiki/xacro">
-    <!--This xacro block sets and loads the depth camera for the robot.
-        Multiple cameras can be placed under the drum arms to assist with digging operations. -->
-        <!-- This doesn't end up being the camera spawned in the simulation, i never got it to work,
-            the camera shown is in the rerassor.xacro.urdf file  -->
-    <xacro:macro name="rerassor_camera" params="camera_prefix">
-        <xacro:property name="cameraSize" value="0.01"/>
-        <xacro:property name="cameraMass" value="0.1"/>
-        <link name="${camera_prefix}">
+<robot name="ezrassor" xmlns:xacro="http://www.ros.org/wiki/xacro">
+    <!-- Macro to add a depth camera to a given parent link -->
+    <xacro:macro name="ezrassor_camera" params="camera_prefix parent x y z">
+        <!-- Camera link and fixed optical frame -->
+        <link name="${camera_prefix}_link">
+            <inertial>
+                <origin xyz="0 0 0" rpy="0 0 0"/>
+                <mass value="${cameraMass}"/>
+                <inertia ixx="0.0001" iyy="0.0001" izz="0.0001" ixy="0" ixz="0" iyz="0"/>
+            </inertial>
             <collision>
                 <origin xyz="0 0 0" rpy="0 0 0"/>
@@ -23,60 +23,20 @@
                 <material name="green"/>
             </visual>
-            <inertial>
-                <mass value="${cameraMass}" />
-                <origin xyz="0 0 0" rpy="0 0 0"/>
-                <xacro:box_inertia m="${cameraMass}" x="${cameraSize}" y="${cameraSize}" z="${cameraSize}" />
-                <inertia ixx="1e-6" ixy="0" ixz="0" iyy="1e-6" iyz="0" izz="1e-6" />
-            </inertial>
+        </link>
+        <link name="${camera_prefix}_optical">
+            <!-- no inertial, collision or visual: purely optical frame -->
         </link>
         <joint name="${camera_prefix}_joint" type="fixed">
-            <origin xyz=".3 0 -.1" rpy="0 0 0"/>
-            <axis xyz="0 1 0" />
-            <parent link="base_link"/>
-            <child link="depth_camera_front"/>
+            <parent link="${parent}"/>
+            <child link="${camera_prefix}_link"/>
+            <origin xyz="${x} ${y} ${z}" rpy="0 0 0"/>
         </joint>
-        <gazebo reference="${camera_prefix}">
-            <sensor name="${camera_prefix}_sensor" type="depth">
-                <always_on>0</always_on>
-                <update_rate>1</update_rate>
-                <camera name="${camera_prefix}_depth_camera">
-                    <horizontal_fov>1.29154</horizontal_fov>
-                    <image>
-                        <width>640</width>
-                        <height>480</height>
-                    </image>
-                    <clip>
-                        <near>0.105</near>
-                        <far>10</far>
-                    </clip>
-                    <distortion>
-                        <k1>0.1</k1>
-                        <k2>0.2</k2>
-                        <k3>0.3</k3>
-                        <p1>0.4</p1>
-                        <p2>0.5</p2>
-                        <center>0.5 0.5</center>
-                    </distortion>
-                </camera>
-                <plugin name="${camera_prefix}_controller" filename="libgazebo_ros_camera.so">
-                    <ros>
-                        <remapping>custom_camera/image_raw:=color/image_raw</remapping>
-                        <remapping>custom_camera/image_depth:=depth/image_raw</remapping>
-                        <remapping>custom_camera/camera_info_depth:=depth/camera_info</remapping>
-                        <remapping>custom_camera/points:=depth/points</remapping>
-                    </ros>
-                    <camera_name>front_camera</camera_name>
-                    <frame_name>depth_camera_front</frame_name>
-                    <hack_baseline>0.07</hack_baseline>
-                    <min_depth>0.001</min_depth>
-                </plugin>
-            </sensor>
-        </gazebo>
-        <joint name="depth_camera_optical_joint" type="fixed">
-            <origin xyz="0 0 0" rpy="${-pi/2} 0 ${-pi/2}"/>
-            <parent link="depth_camera_front"/>
-            <child link="depth_camera_optical_frame"/>
+        <joint name="${camera_prefix}_optical_joint" type="fixed">
+            <parent link="${camera_prefix}_link"/>
+            <child link="${camera_prefix}_optical"/>
+            <!-- Rotate optical frame: +Z forward, +X right, +Y down -->
+            <origin xyz="0 0 0" rpy="-1.5708 0 -1.5708"/>
         </joint>
-        <link name="depth_camera_optical_frame"/>
+        <!-- Gazebo sensor is defined in the main URDF to ensure it attaches to the optical link -->
     </xacro:macro>
 </robot>

File: rover_ros2/rover_description/urdf/imu.xacro (robot description, xacro)
@@ -1,43 +1,32 @@
 <?xml version='1.0'?>
-<robot name="rerassor"
-    xmlns:xacro="http://www.ros.org/wiki/xacro">
-    <!--This xacro block sets a new imu (inertial measurement unit) for the robot.
-        Inputs:
-            imu_prefix: the name that will be used to reference this imu
-            imua_size: float value representing the size of the imu
-            imu_mass: float value representing the mass of the imu
-            front_facing: [true/false] represent whether or not the drum is front facing
-            link_origin: an origin tag representing the xyz,rpy for the drum link
-    -->
-    <xacro:macro name="imu" params="imu_prefix camera_size camera_mass *joint_origin">
-    	<link name="${imu_prefix}">
-    		<collision>
-    			<origin xyz="0 0 0" rpy="0 0 0"/>
-    			<geometry>
-    				<box size="${camera_size} ${camera_size} ${camera_size}"/>
-    			</geometry>
-    		</collision>
-    		<visual>
-    			<origin xyz="0 0 0" rpy="0 0 0"/>
-    			<geometry>
-    				<box size="${camera_size} ${camera_size} ${camera_size}"/>
-    			</geometry>
-    			<material name="green"/>
-    		</visual>
-    		<inertial>
-    			<mass value="${camera_mass}" />
-    			<origin xyz="0 0 0" rpy="0 0 0"/>
-    			<xacro:box_inertia m="${camera_mass}" x="${camera_size}" y="${camera_size}" z="${camera_size}" />
-    			<inertia ixx="1e-6" ixy="0" ixz="0" iyy="1e-6" iyz="0" izz="1e-6" />
-    		</inertial>
-    	</link>
-    	<joint name="${imu_prefix}_joint" type="fixed">
-            <xacro:insert_block name="joint_origin"/>
-    		<axis xyz="0 0 0" />
-    		<parent link="base_link"/>
-    		<child link="${imu_prefix}"/>
-    	</joint>
-        <gazebo reference="${imu_prefix}">
-            <gravity>true</gravity>
+<robot name="ezrassor" xmlns:xacro="http://www.ros.org/wiki/xacro">
+    <!-- Macro to add an IMU sensor to a given parent link -->
+    <xacro:macro name="ezrassor_imu" params="imu_prefix parent xyz rpy">
+        <link name="${imu_prefix}_link">
+            <inertial>
+                <origin xyz="0 0 0" rpy="0 0 0"/>
+                <mass value="0.001"/>
+                <inertia ixx="1e-6" iyy="1e-6" izz="1e-6" ixy="0" ixz="0" iyz="0"/>
+            </inertial>
+            <collision>
+                <origin xyz="0 0 0" rpy="0 0 0"/>
+                <geometry>
+                    <box size="${camera_size} ${camera_size} ${camera_size}"/>
+                </geometry>
+            </collision>
+            <visual>
+                <origin xyz="0 0 0" rpy="0 0 0"/>
+                <geometry>
+                    <box size="${camera_size} ${camera_size} ${camera_size}"/>
+                </geometry>
+                <material name="green"/>
+            </visual>
+        </link>
+        <joint name="${imu_prefix}_joint" type="fixed">
+            <parent link="${parent}"/>
+            <child link="${imu_prefix}_link"/>
+            <origin xyz="${xyz}" rpy="${rpy}"/>
+        </joint>
+        <gazebo reference="${imu_prefix}_link">
             <sensor name="${imu_prefix}_sensor" type="imu">
                 <always_on>true</always_on>
@@ -45,13 +34,5 @@
                 <visualize>true</visualize>
                 <topic>data</topic>
-                <plugin filename="libgazebo_ros_imu_sensor.so" name="imu_plugin">
-                    <topicName>imu</topicName>
-                    <bodyName>${imu_prefix}</bodyName>
-                    <updateRateHZ>10.0</updateRateHZ>
-                    <gaussianNoise>2.89e-08</gaussianNoise>
-                    <xyzOffset>0 0 0</xyzOffset>
-                    <rpyOffset>0 0 0</rpyOffset>
-                </plugin>
-                <pose>0 0 0 0 0 0</pose>
+                <!-- (Gazebo ROS IMU plugin removed for Gazebo Sim compatibility) -->
             </sensor>
         </gazebo>

File: rover_ros2/rover_description/urdf/paver.xacro (robot description, xacro)
@@ -1,38 +1,39 @@
 <?xml version='1.0'?>
 <robot name="paver" xmlns:xacro="http://www.ros.org/wiki/xacro">
-  <xacro:property name="paverSize" value="0.01"/>
-  <xacro:property name="paverMass" value="1"/>
-  <link name="paver_link">
-    <visual name="paver_visual">
-      <origin xyz="0 0 0" rpy="0 0 0"/>
-      <geometry>
-        <mesh filename="file://meshes/paver.dae" scale="0.01 0.01 0.01"/>
-      </geometry>
-    </visual>
-    <collision name="paver_collision">
-      <origin xyz="0 0 0" rpy="0 0 0"/>
-      <geometry>
-        <mesh filename="file://meshes/paver.dae" scale="0.01 0.01 0.01"/>
-      </geometry>
-      <surface>
-        <friction>
-          <mu>0.5</mu>
-          <mu2>0.5</mu2>
-        </friction>
-      </surface>
-    </collision>
-    <inertial>
-      <origin xyz="0 0 0" rpy="0 0 0"/>
-      <mass value="${paverMass}"/>
-      <inertia ixx="0.329" ixy="0" ixz="0" iyy="0.329" iyz="0" izz="0.625"/>
-    </inertial>
-  </link>
-  <gazebo reference="paver_link">
-    <selfCollide>1</selfCollide>
-    <mu1 value="0.5"/>
-    <mu2 value="0.5"/>
-    <kp value="10000000.0" />
-    <kd value="1.0" />
-    <fdir1 value="1 0 0"/>
-  </gazebo>
+    <xacro:property name="paverSize" value="0.01"/>
+    <xacro:property name="paverMass" value="1"/>
+    <link name="paver_link">
+        <inertial>
+            <origin xyz="0 0 0" rpy="0 0 0"/>
+            <xacro:call macro="cylinder_inertia" m="${paverMass}" r="0.955" h="0.275"/>
+        </inertial>
+        <visual name="paver_visual">
+            <origin xyz="0 0 0" rpy="0 0 0"/>
+            <geometry>
+                <cylinder radius="0.955" length="0.275"/>
+            </geometry>
+        </visual>
+        <collision name="paver_collision">
+            <origin xyz="0 0 0" rpy="0 0 0"/>
+            <geometry>
+                <cylinder radius="0.955" length="0.275"/>
+            </geometry>
+            <surface>
+                <friction>
+                    <mu>0.5</mu>
+                    <mu2>0.5</mu2>
+                </friction>
+            </surface>
+        </collision>
+    </link>
+    <!-- Paver is attached via a hinge to the base_link in the main URDF -->
+    <xacro:macro name="paver" params="">
+        <joint name="paver_hinge_joint" type="revolute">
+            <origin xyz="0 1.2 0" rpy="0 0 0"/>
+            <parent link="base_link"/>
+            <child link="paver_link"/>
+            <axis xyz="1 0 0"/>
+            <limit lower="0" upper="1.57" effort="50" velocity="1.0"/>
+        </joint>
+    </xacro:macro>
 </robot>
