Commit message: updated xacros to not use meshes and use gazebo harmonic

File: rover_ros2/rover_description/urdf/rerassor.urdf.xacro (robot description, xacro)
@@ -1,242 +1,209 @@
 <?xml version='1.0'?>
-<robot name="rerassor" xmlns:xacro="http://www.ros.org/wiki/xacro">
-	<xacro:property name="cameraSize" value="0.01"/>
-	<xacro:property name="cameraMass" value="0.1"/>
-    <xacro:include filename="macros.xacro" />
-	<xacro:include filename="materials.xacro" />
-	<xacro:include filename="imu.xacro" />
-	<!--Camera x y z values guesstimated to align with the mast-->
-	 <joint name="camera_optical_joint" type="fixed">
-		<origin xyz="1.8 0 3.7" rpy="0 0 0" />
-        <parent link="base_link" />
-        <child link="camera_link_optical" />
-    </joint>
-    <link name="camera_link_optical"></link>
-	<gazebo reference="camera_link_optical">
-        <sensor type="camera" name="my_camera">
-			<always_on>0</always_on>
+<robot name="ezrassor" xmlns:xacro="http://www.ros.org/wiki/xacro">
+    <xacro:property name="cameraSize" value="0.01"/>
+    <xacro:property name="cameraMass" value="0.1"/>
+    <xacro:include filename="$(find ezrassor_sim_description)/urdf/macros.xacro" />
+    <xacro:include filename="$(find ezrassor_sim_description)/urdf/materials.xacro" />
+    <xacro:include filename="$(find ezrassor_sim_description)/urdf/imu.xacro" />
+    <!-- Camera position guesstimated to align with the mast -->
+    <xacro:property name="camera_x" value="0.0"/>
+    <xacro:property name="camera_y" value="0.3"/>
+    <xacro:property name="camera_z" value="1.5"/>
+    <!-- Base link (main body) -->
+    <link name="base_link">
+        <inertial>
+            <origin xyz="0 0 0" rpy="0 0 0"/>
+            <!-- Using box inertia approximation for main body -->
+            <xacro:call macro="box_inertia" m="50" x="1.0" y="1.5" z="0.3"/>
+        </inertial>
+        <collision name='base_link_collision'>
+            <origin xyz="0 0 0" rpy="0 0 0"/>
+            <geometry>
+                <box size="2.058 4.327 2.917"/>
+            </geometry>
+            <!-- Surface properties -->
+            <surface>
+                <friction>
+                    <mu>0.5</mu>
+                    <mu2>0.5</mu2>
+                </friction>
+                <contact>
+                    <kp>100000.0</kp>
+                    <kd>1.0</kd>
+                </contact>
+            </surface>
+        </collision>
+        <visual name='base_link_visual'>
+            <origin xyz="0 0 0" rpy="0 0 0"/>
+            <geometry>
+                <box size="2.058 4.327 2.917"/>
+            </geometry>
+            <material name="yellow"><color rgba="0.973 0.953 0.208 1"/></material>
+        </visual>
+    </link>
+    <!-- Base link is root of the robot -->
+    <joint name="base_link_fixed" type="fixed">
+        <parent link="world"/>
+        <child link="base_link"/>
+    </joint>
+    <!-- Four Wheels attached to base_link -->
+    <!-- Left Front Wheel -->
+    <link name="left_wheel_front_link">
+        <inertial>
+            <origin xyz="0 0 0" rpy="0 0 0"/>
+            <xacro:call macro="cylinder_inertia" m="5" r="0.18" h="0.2"/>
+        </inertial>
+        <collision name="left_wheel_front_collision">
+            <origin xyz="0 0 0" rpy="0 0 0"/>
+            <geometry>
+                <cylinder radius="0.18" length="0.2"/>
+            </geometry>
+            <surface>
+                <friction>
+                    <mu>1.5</mu>
+                    <mu2>1.5</mu2>
+                </friction>
+            </surface>
+        </collision>
+        <visual name="left_wheel_front_visual">
+            <origin xyz="0 0 0" rpy="0 0 0"/>
+            <geometry>
+                <cylinder radius="0.18" length="0.2"/>
+            </geometry>
+        </visual>
+    </link>
+    <joint name="left_wheel_front_joint" type="continuous">
+        <origin xyz="-0.9 1.0 -0.2" rpy="0 0 0"/>
+        <parent link="base_link"/>
+        <child link="left_wheel_front_link"/>
+        <axis xyz="0 1 0"/>
+        <limit effort="1000.0" velocity="5.0"/>
+    </joint>
+    <!-- Right Front Wheel -->
+    <link name="right_wheel_front_link">
+        <inertial>
+            <origin xyz="0 0 0" rpy="0 0 0"/>
+            <xacro:call macro="cylinder_inertia" m="5" r="0.18" h="0.2"/>
+        </inertial>
+        <collision name="right_wheel_front_collision">
+            <origin xyz="0 0 0" rpy="0 0 0"/>
+            <geometry>
+                <cylinder radius="0.18" length="0.2"/>
+            </geometry>
+            <surface>
+                <friction>
+                    <mu>1.5</mu>
+                    <mu2>1.5</mu2>
+                </friction>
+            </surface>
+        </collision>
+        <visual name="right_wheel_front_visual">
+            <origin xyz="0 0 0" rpy="0 0 0"/>
+            <geometry>
+                <cylinder radius="0.18" length="0.2"/>
+            </geometry>
+        </visual>
+    </link>
+    <joint name="right_wheel_front_joint" type="continuous">
+        <origin xyz="0.9 1.0 -0.2" rpy="0 0 0"/>
+        <parent link="base_link"/>
+        <child link="right_wheel_front_link"/>
+        <axis xyz="0 1 0"/>
+        <limit effort="1000.0" velocity="5.0"/>
+    </joint>
+    <!-- Left Back Wheel -->
+    <link name="left_wheel_back_link">
+        <inertial>
+            <origin xyz="0 0 0" rpy="0 0 0"/>
+            <xacro:call macro="cylinder_inertia" m="5" r="0.18" h="0.2"/>
+        </inertial>
+        <collision name="left_wheel_back_collision">
+            <origin xyz="0 0 0" rpy="0 0 0"/>
+            <geometry>
+                <cylinder radius="0.18" length="0.2"/>
+            </geometry>
+            <surface>
+                <friction>
+                    <mu>1.5</mu>
+                    <mu2>1.5</mu2>
+                </friction>
+            </surface>
+        </collision>
+        <visual name="left_wheel_back_visual">
+            <origin xyz="0 0 0" rpy="0 0 0"/>
+            <geometry>
+                <cylinder radius="0.18" length="0.2"/>
+            </geometry>
+        </visual>
+    </link>
+    <joint name="left_wheel_back_joint" type="continuous">
+        <origin xyz="-0.9 -1.0 -0.2" rpy="0 0 0"/>
+        <parent link="base_link"/>
+        <child link="left_wheel_back_link"/>
+        <axis xyz="0 1 0"/>
+        <limit effort="1000.0" velocity="5.0"/>
+    </joint>
+    <!-- Right Back Wheel -->
+    <link name="right_wheel_back_link">
+        <inertial>
+            <origin xyz="0 0 0" rpy="0 0 0"/>
+            <xacro:call macro="cylinder_inertia" m="5" r="0.18" h="0.2"/>
+        </inertial>
+        <collision name="right_wheel_back_collision">
+            <origin xyz="0 0 0" rpy="0 0 0"/>
+            <geometry>
+                <cylinder radius="0.18" length="0.2"/>
+            </geometry>
+            <surface>
+                <friction>
+                    <mu>1.5</mu>
+                    <mu2>1.5</mu2>
+                </friction>
+            </surface>
+        </collision>
+        <visual name="right_wheel_back_visual">
+            <origin xyz="0 0 0" rpy="0 0 0"/>
+            <geometry>
+                <cylinder radius="0.18" length="0.2"/>
+            </geometry>
+        </visual>
+    </link>
+    <joint name="right_wheel_back_joint" type="continuous">
+        <origin xyz="0.9 -1.0 -0.2" rpy="0 0 0"/>
+        <parent link="base_link"/>
+        <child link="right_wheel_back_link"/>
+        <axis xyz="0 1 0"/>
+        <limit effort="1000.0" velocity="5.0"/>
+    </joint>
+    <!-- Paver attachment (compactor plate) -->
+    <xacro:include filename="$(find ezrassor_sim_description)/urdf/paver.xacro" />
+    <xacro:paver/>
+    <!-- Depth camera attachment -->
+    <xacro:include filename="$(find ezrassor_sim_description)/urdf/camera.xacro" />
+    <xacro:ezrassor_camera camera_prefix="depth_camera" parent="base_link"
+                           x="${camera_x}" y="${camera_y}" z="${camera_z}" />
+    <!-- IMU attachment -->
+    <xacro:include filename="$(find ezrassor_sim_description)/urdf/imu.xacro" />
+    <xacro:ezrassor_imu imu_prefix="imu_link" parent="base_link"
+                        xyz="0 0 0.2" rpy="0 0 0" />
+    <!-- Depth camera sensor (Gazebo Sim format) -->
+    <gazebo reference="depth_camera_optical">
+        <sensor name="depth_camera_sensor" type="depth">
+            <always_on>0</always_on>
             <update_rate>1</update_rate>
-            <visualize>true</visualize>
-            <camera name="cam">
+            <camera name="depth_camera">
                 <horizontal_fov>1.29154</horizontal_fov>
                 <image>
-					<width>640</width>
-					<height>480</height>
-                    <format>R8B8G8</format>
+                    <width>640</width>
+                    <height>480</height>
+                    <format>R8G8B8</format>
                 </image>
-				<clip>
-					<near>0.105</near>
-					<far>100</far>
-				</clip>
+                <clip>
+                    <near>0.1</near>
+                    <far>100.0</far>
+                </clip>
             </camera>
-            <plugin name="camera_controller" filename="libgazebo_ros_camera.so">
-                <frame_name>camera_link_optical</frame_name>
-                <hack_baseline>0.07</hack_baseline>
-                <min_depth>0.001</min_depth>
-            </plugin>
+            <visualize>true</visualize>
         </sensor>
     </gazebo>
-	<!-- End camera -->
-	<!--Tags below represent robot links and joints only-->
-	<link name='base_link'>
-		<pose>0 0 0 0 0 0</pose>
-	</link>
-	<link name='body'>
-		<pose>0 0 0 0 0 0</pose>
-		<inertial>
-			<mass value="15.0"/>
-			<origin xyz="0 0 0" rpy=" 0 0 0"/>
-			<inertia ixx="16.67" ixy="0" ixz="0" iyy="16.67" iyz="0" izz="16.67" />
-		</inertial>
-		<collision name='collision'>
-			<origin xyz="0 0 0" rpy=" 0 0 0"/>
-			<geometry>
-       			<mesh filename="file://meshes/base_unit.dae" scale="0.01 0.01 0.01"></mesh>
-			</geometry>
-		</collision>
-		<visual name='base_link_visual'>
-			<origin xyz="0 0 0" rpy=" 0 0 0"/>
-			<geometry>
-        		<mesh filename="file://meshes/base_unit.dae" scale="0.01 0.01 0.01"></mesh>
-			</geometry>
-		</visual>
-	</link>
-    <gazebo reference="base_link">
-		<material>Gazebo/ZincYellow</material>
-		<selfCollide>0</selfCollide>
-    </gazebo>
-    <joint name="body_joint" type="fixed">
-		<axis xyz="0 0 0"/>
-		<origin xyz="0 0 1.0" rpy="0 0 0"/>
-		<parent link="base_link"/>
-		<child link="body"/>
-	</joint>
-	<!-- Define wheels directly (formerly macros) -->
-	<!-- Left Front Wheel -->
-    <!---->
-	<link name="left_wheel_front_link">
-		<visual name="left_wheel_front_visual">
-			<origin xyz="0 0 0" rpy="0 0 0"/>
-			<geometry>
-				<mesh filename="file://meshes/wheel.dae" scale="0.01 0.01 0.01"/>
-			</geometry>
-		</visual>
-		<collision name="collision">
-			<origin xyz="0 0 0" rpy="0 0 0"/>
-			<geometry>
-				<mesh filename="file://meshes/wheel.dae" scale="0.01 0.01 0.01"/>
-			</geometry>
-			<surface>
-				<friction>
-					<mu>0.5</mu>
-					<mu2>0.5</mu2>
-				</friction>
-			</surface>
-		</collision>
-		 <inertial>
-			<origin xyz="0 0 0" rpy="0 0 0"/>
-			<mass value="5"/>
-			<inertia ixx="0.329" ixy="0" ixz="0" iyy="0.329" iyz="0" izz="0.625"/>
-		</inertial>
-	</link>
-	<joint name="left_wheel_front_joint" type="continuous">
-		<origin xyz="1.5 1.2 0.2" rpy="${pi/2} 0 0"/>
-		<child link="left_wheel_front_link"/>
-		<parent link="body"/>
-		<axis xyz="0 0 -1"/>
-		<dynamics damping="0.5"/>
-	</joint>
-	<gazebo reference="left_wheel_front_link">
-		<selfCollide>1</selfCollide>
-		<mu1 value="0.5"/>
-		<mu2 value="0.5"/>
-		<kp value="10000000.0" />
-		<kd value="1.0" />
-		<fdir1 value="1 0 0"/>
-	</gazebo>
-	<link name="right_wheel_front_link">
-		<visual name="right_wheel_front_visual">
-			<origin xyz="0 0 0" rpy="0 0 0"/>
-			<geometry>
-				<mesh filename="file://meshes/wheel.dae" scale="0.01 0.01 0.01"/>
-			</geometry>
-		</visual>
-		<collision name="collision">
-			<origin xyz="0 0 0" rpy="0 0 0"/>
-			<geometry>
-				<mesh filename="file://meshes/wheel.dae" scale="0.01 0.01 0.01"/>
-			</geometry>
-			<surface>
-				<friction>
-					<mu>0.5</mu>
-					<mu2>0.5</mu2>
-				</friction>
-			</surface>
-		</collision>
-		<inertial>
-			<origin xyz="0 0 0" rpy="0 0 0"/>
-			<mass value="5"/>
-			<inertia ixx="0.329" ixy="0" ixz="0" iyy="0.329" iyz="0" izz="0.625"/>
-		</inertial>
-	</link>
-	<joint name="right_wheel_front_joint" type="continuous">
-		<origin xyz="1.5 -1.2 0.2" rpy="${3 * pi / 2} 0 0"/>
-		<child link="right_wheel_front_link"/>
-		<parent link="body"/>
-		<axis xyz="0 0 1"/>
-		<dynamics damping="0.5"/>
-	</joint>
-	<gazebo reference="right_wheel_front_link">
-		<selfCollide>1</selfCollide>
-		<mu1 value="0.5"/>
-		<mu2 value="0.5"/>
-		<kp value="10000000.0" />
-		<kd value="1.0" />
-		<fdir1 value="1 0 0"/>
-	</gazebo>
-	<link name="right_wheel_back_link">
-		<visual name="right_back_front_visual">
-			<origin xyz="0 0 0" rpy="0 0 0"/>
-			<geometry>
-				<mesh filename="file://meshes/wheel.dae" scale="0.01 0.01 0.01"/>
-			</geometry>
-		</visual>
-		<collision name="collision">
-			<origin xyz="0 0 0" rpy="0 0 0"/>
-			<geometry>
-				<mesh filename="file://meshes/wheel.dae" scale="0.01 0.01 0.01"/>
-			</geometry>
-			<surface>
-				<friction>
-					<mu>0.5</mu>
-					<mu2>0.5</mu2>
-				</friction>
-			</surface>
-		</collision>
-		<inertial>
-			<origin xyz="0 0 0" rpy="0 0 0"/>
-			<mass value="5"/>
-			<inertia ixx="0.329" ixy="0" ixz="0" iyy="0.329" iyz="0" izz="0.625"/>
-		</inertial>
-	</link>
-	<joint name="right_wheel_back_joint" type="continuous">
-		<origin xyz="-1.5 -1.2 0.2" rpy="${3 * pi / 2} 0 0"/>
-		<child link="right_wheel_back_link"/>
-		<parent link="body"/>
-		<axis xyz="0 0 1"/>
-		<dynamics damping="0.5"/>
-	</joint>
-	<gazebo reference="right_wheel_back_link">
-		<selfCollide>1</selfCollide>
-		<mu1 value="0.5"/>
-		<mu2 value="0.5"/>
-		<kp value="10000000.0" />
-		<kd value="1.0" />
-		<fdir1 value="1 0 0"/>
-	</gazebo>
-	<link name="left_wheel_back_link">
-		<visual name="left_back_front_visual">
-			<origin xyz="0 0 0" rpy="0 0 0"/>
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
File: rover_ros2/rover_description/urdf/wheel.xacro (robot description, xacro)
@@ -1,54 +1,40 @@
 <?xml version='1.0'?>
-<robot name="rerassor"
-    xmlns:xacro="http://www.ros.org/wiki/xacro">
+<robot name="ezrassor" xmlns:xacro="http://www.ros.org/wiki/xacro">
+    <!-- Macro defining the wheel geometry (cylinder) -->
     <xacro:macro name="wheel_mesh">
-        <mesh filename="file://$(find rerassor_sim_description)/meshes/wheel.dae" scale="0.35 0.35 0.35"></mesh>
+        <cylinder radius="0.18" length="0.2"/>
     </xacro:macro>
-    <!--This xacro block sets a new driving wheel for the robot.
-        Inputs:
-            wheel_prefix: the name that will be used to reference this wheel
-            yaw: the yaw value that will be used for the wheel link
-            joint_origin: an origin tag representing the xyz,rpy for the wheel joint
-    -->
-    <xacro:macro name="rerassor_wheel" params="wheel_prefix yaw *joint_origin">
+    <!-- The wheel module macro (if it were used) -->
+    <xacro:macro name="ezrassor_wheel" params="wheel_prefix parent xyz rpy yaw">
         <link name="${wheel_prefix}">
             <inertial>
-                <origin xyz="0 0 0" rpy="0 0 ${yaw}" />
-                <mass value="5"/>
-                <xacro:cylinder_inertia m="5" r="0.18" h="0.2"/>
+                <origin xyz="0 0 0" rpy="0 0 0"/>
+                <xacro:call macro="cylinder_inertia" m="5" r="0.18" h="0.2"/>
             </inertial>
             <visual name="${wheel_prefix}_visual">
                 <origin xyz="0 0 0" rpy="0 0 ${yaw}"/>
                 <geometry>
-                    <xacro:wheel_mesh />
+                    <xacro:wheel_mesh/>
                 </geometry>
             </visual>
-            <collision name="collision">
+            <collision name="${wheel_prefix}_collision">
                 <origin xyz="0 0 0" rpy="0 0 ${yaw}"/>
                 <geometry>
-                    <xacro:wheel_mesh />
+                    <xacro:wheel_mesh/>
                 </geometry>
                 <surface>
                     <friction>
-                        <mu> 1.5 </mu>
-                        <mu2> 1.5 </mu2>
+                        <mu>1.5</mu>
+                        <mu2>1.5</mu2>
                     </friction>
                 </surface>
             </collision>
         </link>
-        <gazebo reference="${wheel_prefix}">
-            <selfCollide>1</selfCollide>
-            <mu1 value="1.5"/>
-            <mu2 value="1.5"/>
-            <kp value="10000000.0" />
-            <kd value="1.0" />
-            <fdir1 value="1 0 0"/>
-        </gazebo>
         <joint name="${wheel_prefix}_joint" type="continuous">
-            <xacro:insert_block name="joint_origin"/>
+            <origin xyz="${xyz}" rpy="${rpy}"/>
+            <parent link="${parent}"/>
             <child link="${wheel_prefix}"/>
-            <parent link="base_link"/>
-            <axis xyz="0 1 0" rpy="0 0 0"/>
-            <dynamics damping="0.2"/>
+            <axis xyz="0 1 0"/>
+            <limit effort="1000" velocity="5"/>
         </joint>
     </xacro:macro>

Commit message: renamed all mentions of ezrassor to rerassor

File: rover_ros2/rover_description/urdf/camera.xacro (robot description, xacro)
@@ -1,6 +1,6 @@
 <?xml version='1.0'?>
-<robot name="ezrassor" xmlns:xacro="http://www.ros.org/wiki/xacro">
+<robot name="rerassor" xmlns:xacro="http://www.ros.org/wiki/xacro">
     <!-- Macro to add a depth camera to a given parent link -->
-    <xacro:macro name="ezrassor_camera" params="camera_prefix parent x y z">
+    <xacro:macro name="rerassor_camera" params="camera_prefix parent x y z">
         <!-- Camera link and fixed optical frame -->
         <link name="${camera_prefix}_link">

File: rover_ros2/rover_description/urdf/imu.xacro (robot description, xacro)
@@ -1,6 +1,6 @@
 <?xml version='1.0'?>
-<robot name="ezrassor" xmlns:xacro="http://www.ros.org/wiki/xacro">
+<robot name="rerassor" xmlns:xacro="http://www.ros.org/wiki/xacro">
     <!-- Macro to add an IMU sensor to a given parent link -->
-    <xacro:macro name="ezrassor_imu" params="imu_prefix parent xyz rpy">
+    <xacro:macro name="rerassor_imu" params="imu_prefix parent xyz rpy">
         <link name="${imu_prefix}_link">
             <inertial>

File: rover_ros2/rover_description/urdf/rerassor.urdf.xacro (robot description, xacro)
@@ -1,9 +1,9 @@
 <?xml version='1.0'?>
-<robot name="ezrassor" xmlns:xacro="http://www.ros.org/wiki/xacro">
+<robot name="rerassor" xmlns:xacro="http://www.ros.org/wiki/xacro">
     <xacro:property name="cameraSize" value="0.01"/>
     <xacro:property name="cameraMass" value="0.1"/>
-    <xacro:include filename="$(find ezrassor_sim_description)/urdf/macros.xacro" />
-    <xacro:include filename="$(find ezrassor_sim_description)/urdf/materials.xacro" />
-    <xacro:include filename="$(find ezrassor_sim_description)/urdf/imu.xacro" />
+    <xacro:include filename="$(find rerassor_sim_description)/urdf/macros.xacro" />
+    <xacro:include filename="$(find rerassor_sim_description)/urdf/materials.xacro" />
+    <xacro:include filename="$(find rerassor_sim_description)/urdf/imu.xacro" />
     <!-- Camera position guesstimated to align with the mast -->
     <xacro:property name="camera_x" value="0.0"/>
@@ -177,13 +177,13 @@
     </joint>
     <!-- Paver attachment (compactor plate) -->
-    <xacro:include filename="$(find ezrassor_sim_description)/urdf/paver.xacro" />
+    <xacro:include filename="$(find rerassor_sim_description)/urdf/paver.xacro" />
     <xacro:paver/>
     <!-- Depth camera attachment -->
-    <xacro:include filename="$(find ezrassor_sim_description)/urdf/camera.xacro" />
-    <xacro:ezrassor_camera camera_prefix="depth_camera" parent="base_link"
+    <xacro:include filename="$(find rerassor_sim_description)/urdf/camera.xacro" />
+    <xacro:rerassor_camera camera_prefix="depth_camera" parent="base_link"
                            x="${camera_x}" y="${camera_y}" z="${camera_z}" />
     <!-- IMU attachment -->
-    <xacro:include filename="$(find ezrassor_sim_description)/urdf/imu.xacro" />
-    <xacro:ezrassor_imu imu_prefix="imu_link" parent="base_link"
+    <xacro:include filename="$(find rerassor_sim_description)/urdf/imu.xacro" />
+    <xacro:rerassor_imu imu_prefix="imu_link" parent="base_link"
                         xyz="0 0 0.2" rpy="0 0 0" />
     <!-- Depth camera sensor (Gazebo Sim format) -->

File: rover_ros2/rover_description/urdf/wheel.xacro (robot description, xacro)
@@ -1,4 +1,4 @@
 <?xml version='1.0'?>
-<robot name="ezrassor" xmlns:xacro="http://www.ros.org/wiki/xacro">
+<robot name="rerassor" xmlns:xacro="http://www.ros.org/wiki/xacro">
     <!-- Macro defining the wheel geometry (cylinder) -->
     <xacro:macro name="wheel_mesh">
@@ -6,5 +6,5 @@
     </xacro:macro>
     <!-- The wheel module macro (if it were used) -->
-    <xacro:macro name="ezrassor_wheel" params="wheel_prefix parent xyz rpy yaw">
+    <xacro:macro name="rerassor_wheel" params="wheel_prefix parent xyz rpy yaw">
         <link name="${wheel_prefix}">
             <inertial>
