Commit message: mesh based urdf rendering properly with rivz2 config

File: rover_ros2/rover_description/urdf/camera.xacro (robot description, xacro)
@@ -1,13 +1,13 @@
 <?xml version='1.0'?>
-<robot name="rerassor" xmlns:xacro="http://www.ros.org/wiki/xacro">
-    <!-- Macro to add a depth camera to a given parent link -->
-    <xacro:macro name="rerassor_camera" params="camera_prefix parent x y z">
-        <!-- Camera link and fixed optical frame -->
-        <link name="${camera_prefix}_link">
-            <inertial>
-                <origin xyz="0 0 0" rpy="0 0 0"/>
-                <mass value="${cameraMass}"/>
-                <inertia ixx="0.0001" iyy="0.0001" izz="0.0001" ixy="0" ixz="0" iyz="0"/>
-            </inertial>
+<robot name="rerassor"
+    xmlns:xacro="http://www.ros.org/wiki/xacro">
+    <!--This xacro block sets and loads the depth camera for the robot.
+        Multiple cameras can be placed under the drum arms to assist with digging operations. -->
+        <!-- This doesn't end up being the camera spawned in the simulation, i never got it to work,
+            the camera shown is in the rerassor.xacro.urdf file  -->
+    <xacro:macro name="rerassor_camera" params="camera_prefix">
+        <xacro:property name="cameraSize" value="0.01"/>
+        <xacro:property name="cameraMass" value="0.1"/>
+        <link name="${camera_prefix}">
             <collision>
                 <origin xyz="0 0 0" rpy="0 0 0"/>
@@ -23,20 +23,60 @@
                 <material name="green"/>
             </visual>
-        </link>
-        <link name="${camera_prefix}_optical">
-            <!-- no inertial, collision or visual: purely optical frame -->
+            <inertial>
+                <mass value="${cameraMass}" />
+                <origin xyz="0 0 0" rpy="0 0 0"/>
+                <xacro:box_inertia m="${cameraMass}" x="${cameraSize}" y="${cameraSize}" z="${cameraSize}" />
+                <inertia ixx="1e-6" ixy="0" ixz="0" iyy="1e-6" iyz="0" izz="1e-6" />
+            </inertial>
         </link>
         <joint name="${camera_prefix}_joint" type="fixed">
-            <parent link="${parent}"/>
-            <child link="${camera_prefix}_link"/>
-            <origin xyz="${x} ${y} ${z}" rpy="0 0 0"/>
+            <origin xyz=".3 0 -.1" rpy="0 0 0"/>
+            <axis xyz="0 1 0" />
+            <parent link="base_link"/>
+            <child link="depth_camera_front"/>
         </joint>
-        <joint name="${camera_prefix}_optical_joint" type="fixed">
-            <parent link="${camera_prefix}_link"/>
-            <child link="${camera_prefix}_optical"/>
-            <!-- Rotate optical frame: +Z forward, +X right, +Y down -->
-            <origin xyz="0 0 0" rpy="-1.5708 0 -1.5708"/>
+        <gazebo reference="${camera_prefix}">
+            <sensor name="${camera_prefix}_sensor" type="depth">
+                <always_on>0</always_on>
+                <update_rate>1</update_rate>
+                <camera name="${camera_prefix}_depth_camera">
+                    <horizontal_fov>1.29154</horizontal_fov>
+                    <image>
+                        <width>640</width>
+                        <height>480</height>
+                    </image>
+                    <clip>
+                        <near>0.105</near>
+                        <far>10</far>
+                    </clip>
+                    <distortion>
+                        <k1>0.1</k1>
+                        <k2>0.2</k2>
+                        <k3>0.3</k3>
+                        <p1>0.4</p1>
+                        <p2>0.5</p2>
+                        <center>0.5 0.5</center>
+                    </distortion>
+                </camera>
+                <plugin name="${camera_prefix}_controller" filename="libgazebo_ros_camera.so">
+                    <ros>
+                        <remapping>custom_camera/image_raw:=color/image_raw</remapping>
+                        <remapping>custom_camera/image_depth:=depth/image_raw</remapping>
+                        <remapping>custom_camera/camera_info_depth:=depth/camera_info</remapping>
+                        <remapping>custom_camera/points:=depth/points</remapping>
+                    </ros>
+                    <camera_name>front_camera</camera_name>
+                    <frame_name>depth_camera_front</frame_name>
+                    <hack_baseline>0.07</hack_baseline>
+                    <min_depth>0.001</min_depth>
+                </plugin>
+            </sensor>
+        </gazebo>
+        <joint name="depth_camera_optical_joint" type="fixed">
+            <origin xyz="0 0 0" rpy="${-pi/2} 0 ${-pi/2}"/>
+            <parent link="depth_camera_front"/>
+            <child link="depth_camera_optical_frame"/>
         </joint>
-        <!-- Gazebo sensor is defined in the main URDF to ensure it attaches to the optical link -->
+        <link name="depth_camera_optical_frame"/>
     </xacro:macro>
 </robot>

File: rover_ros2/rover_description/urdf/wheel.xacro (robot description, xacro)
@@ -1,28 +1,53 @@
 <?xml version='1.0'?>
-<robot name="rerassor" xmlns:xacro="http://www.ros.org/wiki/xacro">
-    <!-- wheel.xacro -->
-    <xacro:macro name="wheel" params="wheel_name parent_link radius width mass origin_xyz origin_rpy">
-        <link name="${wheel_name}_link">
+<robot name="rerassor"
+    xmlns:xacro="http://www.ros.org/wiki/xacro">
+    <xacro:macro name="wheel_mesh">
+        <mesh filename="file://$(find rover_description)/meshes/wheel.dae" scale="0.35 0.35 0.35"></mesh>
+    </xacro:macro>
+    <!--This xacro block sets a new driving wheel for the robot.
+        Inputs:
+            wheel_prefix: the name that will be used to reference this wheel
+            yaw: the yaw value that will be used for the wheel link
+            joint_origin: an origin tag representing the xyz,rpy for the wheel joint
+    -->
+    <xacro:macro name="rerassor_wheel" params="wheel_prefix yaw *joint_origin">
+        <link name="${wheel_prefix}">
             <inertial>
-                <origin xyz="0 0 0" rpy="0 0 0"/>
-                <mass value="${mass}"/>
-                <xacro:cylinder_inertia m="${mass}" r="${radius}" h="${width}"/>
+                <origin xyz="0 0 0" rpy="0 0 ${yaw}" />
+                <mass value="5"/>
+                <xacro:cylinder_inertia m="5" r="0.18" h="0.2"/>
             </inertial>
-            <visual>
-                <origin xyz="0 0 0" rpy="0 0 0"/>
-                <geometry><cylinder radius="${radius}" length="${width}"/></geometry>
-                <material name="Grey"/>
+            <visual name="${wheel_prefix}_visual">
+                <origin xyz="0 0 0" rpy="0 0 ${yaw}"/>
+                <geometry>
+                    <xacro:wheel_mesh />
+                </geometry>
             </visual>
-            <collision>
-                <origin xyz="0 0 0" rpy="0 0 0"/>
-                <geometry><cylinder radius="${radius}" length="${width}"/></geometry>
-                <surface><friction><mu>1.5</mu><mu2>1.5</mu2></friction></surface>
+            <collision name="collision">
+                <origin xyz="0 0 0" rpy="0 0 ${yaw}"/>
+                <geometry>
+                    <xacro:wheel_mesh />
+                </geometry>
+                <surface>
+                    <friction>
+                        <mu> 1.5 </mu>
+                        <mu2> 1.5 </mu2>
+                    </friction>
+                </surface>
             </collision>
         </link>
-        <joint name="${wheel_name}_joint" type="continuous">
-            <parent link="${parent_link}"/>
-            <child link="${wheel_name}_link"/>
-            <origin xyz="${origin_xyz}" rpy="${origin_rpy}"/>
-            <axis xyz="0 1 0"/>  <!-- assuming wheel rotates about the Y-axis of arm frame -->
+        <gazebo reference="${wheel_prefix}">
+            <selfCollide>1</selfCollide>
+            <mu1 value="1.5"/>
+            <mu2 value="1.5"/>
+            <kp value="10000000.0" />
+            <kd value="1.0" />
+            <fdir1 value="1 0 0"/>
+        </gazebo>
+        <joint name="${wheel_prefix}_joint" type="continuous">
+            <xacro:insert_block name="joint_origin"/>
+            <child link="${wheel_prefix}"/>
+            <parent link="base_link"/>
+            <axis xyz="0 1 0" rpy="0 0 0"/>
             <dynamics damping="0.2"/>
         </joint>

Commit message: added in missing gazebo stuff

File: rover_ros2/rover_description/urdf/camera.xacro (robot description, xacro)
@@ -1,4 +1,4 @@
 <?xml version="1.0" encoding="utf-8"?>
-<robot name="rerassor" xmlns:xacro="http://www.ros.org/wiki/xacro">
+<robot xmlns:xacro="http://www.ros.org/wiki/xacro">
     <!-- PHYSICAL CAMERA -->
     <link name="camera_link">
@@ -19,5 +19,5 @@
             <origin xyz="0 0 0" rpy="0 0 0" />
             <geometry>
-                <mesh filename="package://rover_description/meshes/B-C.STL" />
+                <mesh filename="package://rover_description/meshes/camera.STL" />
             </geometry>
             <material name="">
@@ -29,5 +29,5 @@
             <origin xyz="0 0 0" rpy="0 0 0" />
             <geometry>
-                <mesh filename="package://rover_description/meshes/B-C.STL" />
+                <mesh filename="package://rover_description/meshes/camera.STL" />
             </geometry>
         </collision>

File: rover_ros2/rover_description/urdf/chassis.xacro (robot description, xacro)
@@ -1,4 +1,4 @@
 <?xml version="1.0" encoding="utf-8"?>
-<robot name="rerassor" xmlns:xacro="http://www.ros.org/wiki/xacro">
+<robot xmlns:xacro="http://www.ros.org/wiki/xacro">
     <link name="chassis_link">
         <inertial>
@@ -29,5 +29,5 @@
             <origin xyz="0 0 0" rpy="0 0 0" />
             <geometry>
-                <mesh filename="package://rover_description/meshes/BASE.STL" />
+                <mesh filename="package://rover_description/meshes/chassis.STL" />
             </geometry>
         </collision>

File: rover_ros2/rover_description/urdf/gazebo.xacro (robot description, xacro)
@@ -1,4 +1,4 @@
 <?xml version="1.0" encoding="utf-8"?>
-<robot name="rerassor" xmlns:xacro="http://www.ros.org/wiki/xacro">
+<robot name="gazebo" xmlns:xacro="http://www.ros.org/wiki/xacro">
     <!-- CHASSIS -->
     <gazebo reference="chassis_link">
@@ -9,13 +9,53 @@
         <material>Gazebo/Gray</material>
     </gazebo>
+    <transmission name="front_left_wheel_transmission">
+        <type>transmission_interface/SimpleTransmission</type>
+        <joint    name="front_left_wheel_joint">
+            <hardwareInterface>velocity</hardwareInterface>
+        </joint>
+        <actuator name="fl_act">
+            <hardwareInterface>velocity</hardwareInterface>
+            <mechanicalReduction>1.0</mechanicalReduction>
+        </actuator>
+    </transmission>
     <gazebo reference="front_right_wheel_link">
         <material>Gazebo/Gray</material>
     </gazebo>
+    <transmission name="front_right_wheel_transmission">
+        <type>transmission_interface/SimpleTransmission</type>
+        <joint    name="front_right_wheel_joint">
+            <hardwareInterface>velocity</hardwareInterface>
+        </joint>
+        <actuator name="fr_act">
+            <hardwareInterface>velocity</hardwareInterface>
+            <mechanicalReduction>1.0</mechanicalReduction>
+        </actuator>
+    </transmission>
     <gazebo reference="rear_left_wheel_link">
         <material>Gazebo/Gray</material>
     </gazebo>
+    <transmission name="rear_left_wheel_transmission">
+        <type>transmission_interface/SimpleTransmission</type>
+        <joint    name="rear_left_wheel_joint">
+            <hardwareInterface>velocity</hardwareInterface>
+        </joint>
+        <actuator name="rl_act">
+            <hardwareInterface>velocity</hardwareInterface>
+            <mechanicalReduction>1.0</mechanicalReduction>
+        </actuator>
+    </transmission>
     <gazebo reference="rear_right_wheel_link">
         <material>Gazebo/Gray</material>
     </gazebo>
+    <transmission name="rear_right_wheel_transmission">
+        <type>transmission_interface/SimpleTransmission</type>
+        <joint    name="rear_right_wheel_joint">
+            <hardwareInterface>velocity</hardwareInterface>
+        </joint>
+        <actuator name="rr_act">
+            <hardwareInterface>velocity</hardwareInterface>
+            <mechanicalReduction>1.0</mechanicalReduction>
+        </actuator>
+    </transmission>
     <!-- CAMERA -->
     <gazebo reference="camera_link">
@@ -46,3 +86,11 @@
         </sensor>
     </gazebo>
+    <!-- ROS2 Control Plugin -->
+    <xacro:if value="$(arg use_ros2_control)">
+        <gazebo>
+            <plugin filename="libgz_ros2_control-system.so" name="gz_ros2_control::GazeboSimROS2ControlPlugin">
+                <parameters>$(find rover_control)/controllers/diff_cont.yaml</parameters>
+            </plugin>
+        </gazebo>
+    </xacro:if>
 </robot>

File: rover_ros2/rover_description/urdf/ros2_control.xacro (robot description, xacro)
@@ -1,4 +1,4 @@
 <?xml version="1.0" encoding="utf-8"?>
-<robot name="rerassor" xmlns:xacro="http://www.ros.org/wiki/xacro">
+<robot name="ros2_control" xmlns:xacro="http://www.ros.org/wiki/xacro">
     <ros2_control name="DiffDriveSystem" type="system">
         <hardware>

File: rover_ros2/rover_description/urdf/wheels.xacro (robot description, xacro)
@@ -1,4 +1,4 @@
 <?xml version="1.0" encoding="utf-8"?>
-<robot name="rerassor" xmlns:xacro="http://www.ros.org/wiki/xacro">
+<robot name="wheels" xmlns:xacro="http://www.ros.org/wiki/xacro">
     <!-- FRONT LEFT WHEEL -->
     <link name="front_left_wheel_link">
@@ -33,22 +33,11 @@
         </collision>
     </link>
-    <joint name="front_left_wheel_joint" type="revolute">
+    <joint name="front_left_wheel_joint" type="continuous">
         <origin
             xyz="0.2863 0 0.11332"
-            rpy="1.5    <origin
-            xyz="0 0 0"
-            rpy="0 0 0" />
-            <geometry>
-            <mesh
-            filename="package://rover_description/meshes/front_left_wheel.STL" />
-            </geometry>708 -0.036526 0" />
+            rpy="1.5708 -0.036526 0" />
         <parent link="chassis_link" />
         <child link="front_left_wheel_link" />
         <axis xyz="0 0 -1" />
-        <limit
-            lower="0"
-            upper="0"
-            effort="0"
-            velocity="0" />
     </joint>
     <!-- FRONT RIGHT WHEEL -->
@@ -84,5 +73,5 @@
         </collision>
     </link>
-    <joint name="front_right_wheel_joint" type="revolute">
+    <joint name="front_right_wheel_joint" type="continuous">
         <origin
             xyz="-0.0058772 0 0.11332"
@@ -91,9 +80,4 @@
         <child link="front_right_wheel_link" />
         <axis xyz="0 0 -1" />
-        <limit
-            lower="0"
-            upper="0"
-            effort="0"
-            velocity="0" />
     </joint>
     <!-- REAR LEFT WHEEL -->
@@ -129,5 +113,5 @@
         </collision>
     </link>
-    <joint name="rear_left_wheel_joint" type="revolute">
+    <joint name="rear_left_wheel_joint" type="continuous">
         <origin
             xyz="-0.0058772 -0.30031 0.11332"
@@ -136,9 +120,4 @@
         <child link="rear_left_wheel_link" />
         <axis xyz="0 0 -1" />
-        <limit
-            lower="0"
-            upper="0"
-            effort="0"
-            velocity="0" />
     </joint>
     <!-- REAR RIGHT WHEEL -->
@@ -160,5 +139,5 @@
             <origin xyz="0 0 0" rpy="0 0 0" />
             <geometry>
-                <mesh filename="package://rover_description/meshes/B-W4.STL" />
+                <mesh filename="package://rover_description/meshes/rear_right_wheel.STL" />
             </geometry>
             <material name="">
@@ -170,9 +149,9 @@
             <origin xyz="0 0 0" rpy="0 0 0" />
             <geometry>
-                <mesh filename="package://rover_description/meshes/B-W4.STL" />
+                <mesh filename="package://rover_description/meshes/rear_right_wheel.STL" />
             </geometry>
         </collision>
     </link>
-    <joint name="rear_right_wheel_joint" type="revolute">
+    <joint name="rear_right_wheel_joint" type="continuous">
         <origin
             xyz="0.2863 -0.30031 0.11332"
@@ -181,9 +160,4 @@
         <child link="rear_right_wheel_link" />
         <axis xyz="0 0 -1" />
-        <limit
-            lower="0"
-            upper="0"
-            effort="0"
-            velocity="0" />
     </joint>
 </robot>

Commit message: fixed mesh file path issue. rover spawns in gazebo now

File: rover_ros2/rover_description/urdf/camera.xacro (robot description, xacro)
@@ -19,5 +19,5 @@
             <origin xyz="0 0 0" rpy="0 0 0" />
             <geometry>
-                <mesh filename="package://rover_description/meshes/camera.STL" />
+                <mesh filename="file://$(find rover_description)/meshes/camera.STL" />
             </geometry>
             <material name="">
@@ -29,5 +29,5 @@
             <origin xyz="0 0 0" rpy="0 0 0" />
             <geometry>
-                <mesh filename="package://rover_description/meshes/camera.STL" />
+                <mesh filename="file://$(find rover_description)/meshes/camera.STL" />
             </geometry>
         </collision>

File: rover_ros2/rover_description/urdf/chassis.xacro (robot description, xacro)
@@ -20,5 +20,5 @@
                 rpy="0 0 0" />
             <geometry>
-                <mesh filename="package://rover_description/meshes/chassis.STL" />
+                <mesh filename="file://$(find rover_description)/meshes/chassis.STL" />
             </geometry>
             <material name="">
@@ -29,5 +29,5 @@
             <origin xyz="0 0 0" rpy="0 0 0" />
             <geometry>
-                <mesh filename="package://rover_description/meshes/chassis.STL" />
+                <mesh filename="file://$(find rover_description)/meshes/chassis.STL" />
             </geometry>
         </collision>

File: rover_ros2/rover_description/urdf/wheels.xacro (robot description, xacro)
@@ -19,5 +19,5 @@
             <origin xyz="0 0 0" rpy="0 0 0" />
             <geometry>
-                <mesh filename="package://rover_description/meshes/Wheel1.STL" />
+                <mesh filename="file://$(find rover_description)/meshes/Wheel1.STL" />
             </geometry>
             <material name="">
@@ -29,5 +29,5 @@
             <origin xyz="0 0 0" rpy="0 0 0" />
             <geometry>
-                <mesh filename="package://rover_description/meshes/Wheel1.STL" />
+                <mesh filename="file://$(find rover_description)/meshes/Wheel1.STL" />
             </geometry>
         </collision>
@@ -59,5 +59,5 @@
             <origin xyz="0 0 0" rpy="0 0 0" />
             <geometry>
-                <mesh filename="package://rover_description/meshes/Wheel2.STL" />
+                <mesh filename="file://$(find rover_description)/meshes/Wheel2.STL" />
             </geometry>
             <material name="">
@@ -69,5 +69,5 @@
             <origin xyz="0 0 0" rpy="0 0 0" />
             <geometry>
-                <mesh filename="package://rover_description/meshes/Wheel2.STL" />
+                <mesh filename="file://$(find rover_description)/meshes/Wheel2.STL" />
             </geometry>
         </collision>
@@ -99,5 +99,5 @@
             <origin xyz="0 0 0" rpy="0 0 0" />
             <geometry>
-                <mesh filename="package://rover_description/meshes/Wheel3.STL" />
+                <mesh filename="file://$(find rover_description)/meshes/Wheel3.STL" />
             </geometry>
             <material name="">
@@ -109,5 +109,5 @@
             <origin xyz="0 0 0" rpy="0 0 0" />
             <geometry>
-                <mesh filename="package://rover_description/meshes/Wheel3.STL" />
+                <mesh filename="file://$(find rover_description)/meshes/Wheel3.STL" />
             </geometry>
         </collision>
@@ -139,5 +139,5 @@
             <origin xyz="0 0 0" rpy="0 0 0" />
             <geometry>
-                <mesh filename="package://rover_description/meshes/Wheel4.STL" />
+                <mesh filename="file://$(find rover_description)/meshes/Wheel4.STL" />
             </geometry>
             <material name="">
@@ -149,5 +149,5 @@
             <origin xyz="0 0 0" rpy="0 0 0" />
             <geometry>
-                <mesh filename="package://rover_description/meshes/Wheel4.STL" />
+                <mesh filename="file://$(find rover_description)/meshes/Wheel4.STL" />
             </geometry>
         </collision>
