Commit message: added scale of 0.2 to rover

File: rover_ros2/rover_description/urdf/rerassor.xacro.urdf (robot description, URDF)
Before this commit: robot rerassor, 7 links, 6 joints
Links:
- link body: mass 15.0 -> ${15.0*scale_mass}; geometry collision mesh filename=file://$(find rover_description)/meshes/base_unit.dae scale=${0.01*robot_scale} ${0.01*robot_scale} ${0.01*robot_scale}; visual mesh filename=file://$(find rover_description)/meshes/base_unit.dae scale=${0.01*robot_scale} ${0.01*robot_scale} ${0.01*robot_scale}
- link left_wheel_back_link: mass 5 -> ${5*scale_mass}; geometry collision mesh filename=file://$(find rover_description)/meshes/wheel.dae scale=${0.01*robot_scale} ${0.01*robot_scale} ${0.01*robot_scale}; visual mesh filename=file://$(find rover_description)/meshes/wheel.dae scale=${0.01*robot_scale} ${0.01*robot_scale} ${0.01*robot_scale}
- link left_wheel_front_link: mass 5 -> ${5*scale_mass}; geometry collision mesh filename=file://$(find rover_description)/meshes/wheel.dae scale=${0.01*robot_scale} ${0.01*robot_scale} ${0.01*robot_scale}; visual mesh filename=file://$(find rover_description)/meshes/wheel.dae scale=${0.01*robot_scale} ${0.01*robot_scale} ${0.01*robot_scale}
- link right_wheel_back_link: mass 5 -> ${5*scale_mass}; geometry collision mesh filename=file://$(find rover_description)/meshes/wheel.dae scale=${0.01*robot_scale} ${0.01*robot_scale} ${0.01*robot_scale}; visual mesh filename=file://$(find rover_description)/meshes/wheel.dae scale=${0.01*robot_scale} ${0.01*robot_scale} ${0.01*robot_scale}
- link right_wheel_front_link: mass 5 -> ${5*scale_mass}; geometry collision mesh filename=file://$(find rover_description)/meshes/wheel.dae scale=${0.01*robot_scale} ${0.01*robot_scale} ${0.01*robot_scale}; visual mesh filename=file://$(find rover_description)/meshes/wheel.dae scale=${0.01*robot_scale} ${0.01*robot_scale} ${0.01*robot_scale}
Joints:
- joint body_joint: axis 0 0 0 -> (none); origin xyz=0 0 1.0 rpy=0 0 0 -> xyz=0 0 ${1.0*robot_scale} rpy=0 0 0
- joint camera_optical_joint: origin xyz=1.8 0 3.7 rpy=0 0 0 -> xyz=${1.8*robot_scale} 0 ${3.7*robot_scale} rpy=0 0 0
- joint left_wheel_back_joint: origin xyz=-1.5 1.2 0.2 rpy=${pi/2} 0 0 -> xyz=${-1.5*robot_scale} ${ 1.2*robot_scale} ${0.2*robot_scale} rpy=${pi/2} 0 0
- joint left_wheel_front_joint: origin xyz=1.5 1.2 0.2 rpy=${pi/2} 0 0 -> xyz=${1.5*robot_scale} ${1.2*robot_scale} ${0.2*robot_scale} rpy=${pi/2} 0 0
- joint right_wheel_back_joint: origin xyz=-1.5 -1.2 0.2 rpy=${3 * pi / 2} 0 0 -> xyz=${-1.5*robot_scale} ${-1.2*robot_scale} ${0.2*robot_scale} rpy=${3*pi/2} 0 0
- joint right_wheel_front_joint: origin xyz=1.5 -1.2 0.2 rpy=${3 * pi / 2} 0 0 -> xyz=${ 1.5*robot_scale} ${-1.2*robot_scale} ${0.2*robot_scale} rpy=${3*pi/2} 0 0

Commit message: prototype hardware control interface implemented and new teensy firmware (no micro ros)

File: rover_ros2/rover_description/urdf/rerassor.xacro.urdf (robot description, URDF)
Before this commit: robot RASSOR URDF WITH MESHES, 6 links, 5 joints
Links:
- removed link BASE
- added link CHASSIS, mass 6.04730235873931; collision mesh filename=package://rover_description/meshes/BASE.STL; visual mesh filename=package://rover_description/meshes/BASE.STL
- added link base_link
- link B-C: geometry collision mesh filename=package://rover_description/meshes/B-C.STL; visual mesh filename=package://rover_description/meshes/B-C.STL
- link B-W1: geometry collision mesh filename=package://rover_description/meshes/B-W1.STL; visual mesh filename=package://rover_description/meshes/B-W1.STL
- link B-W2: geometry collision mesh filename=package://rover_description/meshes/B-W2.STL; visual mesh filename=package://rover_description/meshes/B-W2.STL
- link B-W3: geometry collision mesh filename=package://rover_description/meshes/B-W3.STL; visual mesh filename=package://rover_description/meshes/B-W3.STL
- link B-W4: geometry collision mesh filename=package://rover_description/meshes/B-W4.STL; visual mesh filename=package://rover_description/meshes/B-W4.STL
Joints:
- added joint CHASSIS_joint: type fixed, parent base_link, child CHASSIS, origin xyz=0 0 0 rpy=0 0 0
- joint Camera: parent BASE -> CHASSIS
- joint Wheel 1: parent BASE -> CHASSIS
- joint Wheel 2: parent BASE -> CHASSIS
- joint Wheel 3: parent BASE -> CHASSIS
- joint Wheel 4: parent BASE -> CHASSIS

Commit message: fixed urdf for ros2 control and gazebo and updated launch files

File: rover_ros2/rover_description/urdf/rerassor.xacro.urdf (robot description, URDF)
Before this commit: robot rerassor, 7 links, 6 joints
Links:
- removed link B-C
- removed link B-W1
- removed link B-W2
- removed link B-W3
- removed link B-W4
- removed link CHASSIS
Joints:
- removed joint CHASSIS_joint
- removed joint Camera
- removed joint Wheel 1
- removed joint Wheel 2
- removed joint Wheel 3
- removed joint Wheel 4

Commit message: added use_js_gui parameter to rsp launcher

File: rover_ros2/rover_description/urdf/rerassor.xacro.urdf (robot description, URDF)
Before this commit: robot rerassor, 1 links, 0 joints
Links:
- added link base_footprint
Joints:
- added joint base_joint: type fixed, parent base_link, child base_footprint, origin xyz=0 0 0 rpy=0 0 0

File: rover_ros2/rover_description/urdf/wheels.xacro (robot description, xacro)
@@ -121,4 +121,5 @@
         <axis xyz="0 0 -1" />
     </joint>
+    <!-- TODO: This wheel is dragging a lot and causing the robot to turn while driving straight -->
     <!-- FRONT RIGHT WHEEL -->
     <link name="front_right_wheel_link">
