Commit message: wheels are correct now but not the length of the wheel tubes

File: rover_ros2/rover_description/urdf/wheels.xacro (robot description, xacro)
@@ -41,6 +41,6 @@
         <axis xyz="0 0 -1" />
     </joint>
-    <!-- FRONT RIGHT WHEEL -->
-    <link name="front_right_wheel_link">
+    <!-- REAR LEFT WHEEL -->
+    <link name="rear_left_wheel_link">
         <inertial>
             <origin
@@ -54,44 +54,4 @@
                 iyy="0.014080784493695"
                 iyz="1.4196513069374E-19"
-                izz="0.023364919828031" />
-        </inertial>
-        <visual>
-            <origin xyz="0 0 0" rpy="0 0 0" />
-            <geometry>
-                <mesh filename="package://rover_description/meshes/front_right_wheel.STL" />
-            </geometry>
-            <material name="">
-                <color
-                    rgba="0.792156862745098 0.819607843137255 0.933333333333333 1" />
-            </material>
-        </visual>
-        <collision>
-            <origin xyz="0 0 0" rpy="0 0 0" />
-            <geometry>
-                <mesh filename="package://rover_description/meshes/front_right_wheel.STL" />
-            </geometry>
-        </collision>
-    </link>
-    <joint name="front_right_wheel_joint" type="continuous">
-        <origin
-            xyz="-0.0058772 0 0.11332"
-            rpy="1.5708 -0.51093 0" />
-        <parent link="chassis_link" />
-        <child link="front_right_wheel_link" />
-        <axis xyz="0 0 -1" />
-    </joint>
-    <!-- REAR LEFT WHEEL -->
-    <link name="rear_left_wheel_link">
-        <inertial>
-            <origin
-                xyz="3.46944695195361E-18 -2.77555756156289E-17 -0.0489261260975664"
-                rpy="0 0 0" />
-            <mass value="3.30391410914092" />
-            <inertia
-                ixx="0.0140807844936951"
-                ixy="-2.16840434497101E-19"
-                ixz="-3.98163543484029E-19"
-                iyy="0.0140807844936951"
-                iyz="9.61227061651265E-19"
                 izz="0.023364919828031" />
         </inertial>
@@ -115,6 +75,6 @@
     <joint name="rear_left_wheel_joint" type="continuous">
         <origin
-            xyz="-0.0058772 -0.30031 0.11332"
-            rpy="1.5708 0.20867 -3.1416" />
+            xyz="-0.0058772 0 0.11332"
+            rpy="1.5708 -0.51093 0" />
         <parent link="chassis_link" />
         <child link="rear_left_wheel_link" />
@@ -125,14 +85,14 @@
         <inertial>
             <origin
-            xyz="0 0 -0.0489261260975665"
-            rpy="0 0 0" />
+                xyz="3.46944695195361E-18 -2.77555756156289E-17 -0.0489261260975664"
+                rpy="0 0 0" />
             <mass value="3.30391410914092" />
             <inertia
                 ixx="0.0140807844936951"
                 ixy="-2.16840434497101E-19"
-                ixz="-2.14131782225971E-19"
+                ixz="-3.98163543484029E-19"
                 iyy="0.0140807844936951"
-                iyz="9.51866693857056E-19"
-                izz="0.0233649198280311" />
+                iyz="9.61227061651265E-19"
+                izz="0.023364919828031" />
         </inertial>
         <visual>
@@ -155,9 +115,49 @@
     <joint name="rear_right_wheel_joint" type="continuous">
         <origin
-            xyz="0.2863 -0.30031 0.11332"
-            rpy="1.5708 0.19754 -3.1416" />
+            xyz="-0.0058772 -0.30031 0.11332"
+            rpy="1.5708 0.20867 -3.1416" />
         <parent link="chassis_link" />
         <child link="rear_right_wheel_link" />
         <axis xyz="0 0 -1" />
     </joint>
+    <!-- FRONT RIGHT WHEEL -->
+    <link name="front_right_wheel_link">
+        <inertial>
+            <origin
+            xyz="0 0 -0.0489261260975665"
+            rpy="0 0 0" />
+            <mass value="3.30391410914092" />
+            <inertia
+                ixx="0.0140807844936951"
+                ixy="-2.16840434497101E-19"
+                ixz="-2.14131782225971E-19"
+                iyy="0.0140807844936951"
+                iyz="9.51866693857056E-19"
+                izz="0.0233649198280311" />
+        </inertial>
+        <visual>
+            <origin xyz="0 0 0" rpy="0 0 0" />
+            <geometry>
+                <mesh filename="package://rover_description/meshes/front_right_wheel.STL" />
+            </geometry>
+            <material name="">
+                <color
+                    rgba="0.792156862745098 0.819607843137255 0.933333333333333 1" />
+            </material>
+        </visual>
+        <collision>
+            <origin xyz="0 0 0" rpy="0 0 0" />
+            <geometry>
+                <mesh filename="package://rover_description/meshes/front_right_wheel.STL" />
+            </geometry>
+        </collision>
+    </link>
+    <joint name="front_right_wheel_joint" type="continuous">
+        <origin
+            xyz="0.2863 -0.30031 0.11332"
+            rpy="1.5708 0.19754 -3.1416" />
+        <parent link="chassis_link" />
+        <child link="front_right_wheel_link" />
+        <axis xyz="0 0 -1" />
+    </joint>
 </robot>

Commit message: Revert "wheels are correct now but not the length of the wheel tubes"
This reverts commit 886d605e59156f5f91ffdaa7d8ac2fc3637fc080.

File: rover_ros2/rover_description/urdf/wheels.xacro (robot description, xacro)
@@ -41,6 +41,6 @@
         <axis xyz="0 0 -1" />
     </joint>
-    <!-- REAR LEFT WHEEL -->
-    <link name="rear_left_wheel_link">
+    <!-- FRONT RIGHT WHEEL -->
+    <link name="front_right_wheel_link">
         <inertial>
             <origin
@@ -54,4 +54,44 @@
                 iyy="0.014080784493695"
                 iyz="1.4196513069374E-19"
+                izz="0.023364919828031" />
+        </inertial>
+        <visual>
+            <origin xyz="0 0 0" rpy="0 0 0" />
+            <geometry>
+                <mesh filename="package://rover_description/meshes/front_right_wheel.STL" />
+            </geometry>
+            <material name="">
+                <color
+                    rgba="0.792156862745098 0.819607843137255 0.933333333333333 1" />
+            </material>
+        </visual>
+        <collision>
+            <origin xyz="0 0 0" rpy="0 0 0" />
+            <geometry>
+                <mesh filename="package://rover_description/meshes/front_right_wheel.STL" />
+            </geometry>
+        </collision>
+    </link>
+    <joint name="front_right_wheel_joint" type="continuous">
+        <origin
+            xyz="-0.0058772 0 0.11332"
+            rpy="1.5708 -0.51093 0" />
+        <parent link="chassis_link" />
+        <child link="front_right_wheel_link" />
+        <axis xyz="0 0 -1" />
+    </joint>
+    <!-- REAR LEFT WHEEL -->
+    <link name="rear_left_wheel_link">
+        <inertial>
+            <origin
+                xyz="3.46944695195361E-18 -2.77555756156289E-17 -0.0489261260975664"
+                rpy="0 0 0" />
+            <mass value="3.30391410914092" />
+            <inertia
+                ixx="0.0140807844936951"
+                ixy="-2.16840434497101E-19"
+                ixz="-3.98163543484029E-19"
+                iyy="0.0140807844936951"
+                iyz="9.61227061651265E-19"
                 izz="0.023364919828031" />
         </inertial>
@@ -75,6 +115,6 @@
     <joint name="rear_left_wheel_joint" type="continuous">
         <origin
-            xyz="-0.0058772 0 0.11332"
-            rpy="1.5708 -0.51093 0" />
+            xyz="-0.0058772 -0.30031 0.11332"
+            rpy="1.5708 0.20867 -3.1416" />
         <parent link="chassis_link" />
         <child link="rear_left_wheel_link" />
@@ -85,14 +125,14 @@
         <inertial>
             <origin
-                xyz="3.46944695195361E-18 -2.77555756156289E-17 -0.0489261260975664"
-                rpy="0 0 0" />
+            xyz="0 0 -0.0489261260975665"
+            rpy="0 0 0" />
             <mass value="3.30391410914092" />
             <inertia
                 ixx="0.0140807844936951"
                 ixy="-2.16840434497101E-19"
-                ixz="-3.98163543484029E-19"
+                ixz="-2.14131782225971E-19"
                 iyy="0.0140807844936951"
-                iyz="9.61227061651265E-19"
-                izz="0.023364919828031" />
+                iyz="9.51866693857056E-19"
+                izz="0.0233649198280311" />
         </inertial>
         <visual>
@@ -115,49 +155,9 @@
     <joint name="rear_right_wheel_joint" type="continuous">
         <origin
-            xyz="-0.0058772 -0.30031 0.11332"
-            rpy="1.5708 0.20867 -3.1416" />
+            xyz="0.2863 -0.30031 0.11332"
+            rpy="1.5708 0.19754 -3.1416" />
         <parent link="chassis_link" />
         <child link="rear_right_wheel_link" />
         <axis xyz="0 0 -1" />
     </joint>
-    <!-- FRONT RIGHT WHEEL -->
-    <link name="front_right_wheel_link">
-        <inertial>
-            <origin
-            xyz="0 0 -0.0489261260975665"
-            rpy="0 0 0" />
-            <mass value="3.30391410914092" />
-            <inertia
-                ixx="0.0140807844936951"
-                ixy="-2.16840434497101E-19"
-                ixz="-2.14131782225971E-19"
-                iyy="0.0140807844936951"
-                iyz="9.51866693857056E-19"
-                izz="0.0233649198280311" />
-        </inertial>
-        <visual>
-            <origin xyz="0 0 0" rpy="0 0 0" />
-            <geometry>
-                <mesh filename="package://rover_description/meshes/front_right_wheel.STL" />
-            </geometry>
-            <material name="">
-                <color
-                    rgba="0.792156862745098 0.819607843137255 0.933333333333333 1" />
-            </material>
-        </visual>
-        <collision>
-            <origin xyz="0 0 0" rpy="0 0 0" />
-            <geometry>
-                <mesh filename="package://rover_description/meshes/front_right_wheel.STL" />
-            </geometry>
-        </collision>
-    </link>
-    <joint name="front_right_wheel_joint" type="continuous">
-        <origin
-            xyz="0.2863 -0.30031 0.11332"
-            rpy="1.5708 0.19754 -3.1416" />
-        <parent link="chassis_link" />
-        <child link="front_right_wheel_link" />
-        <axis xyz="0 0 -1" />
-    </joint>
 </robot>

Commit message: joint and link names changed but not file names

File: rover_ros2/rover_description/urdf/wheels.xacro (robot description, xacro)
@@ -41,6 +41,6 @@
         <axis xyz="0 0 -1" />
     </joint>
-    <!-- FRONT RIGHT WHEEL -->
-    <link name="front_right_wheel_link">
+    <!-- REAR LEFT WHEEL -->
+    <link name="rear_left_wheel_link">
         <inertial>
             <origin
@@ -73,14 +73,14 @@
         </collision>
     </link>
-    <joint name="front_right_wheel_joint" type="continuous">
+    <joint name="rear_left_wheel_joint" type="continuous">
         <origin
             xyz="-0.0058772 0 0.11332"
             rpy="1.5708 -0.51093 0" />
         <parent link="chassis_link" />
-        <child link="front_right_wheel_link" />
+        <child link="rear_left_wheel_link" />
         <axis xyz="0 0 -1" />
     </joint>
-    <!-- REAR LEFT WHEEL -->
-    <link name="rear_left_wheel_link">
+    <!-- REAR RIGHT WHEEL -->
+    <link name="rear_right_wheel_link">
         <inertial>
             <origin
@@ -113,14 +113,14 @@
         </collision>
     </link>
-    <joint name="rear_left_wheel_joint" type="continuous">
+    <joint name="rear_right_wheel_joint" type="continuous">
         <origin
             xyz="-0.0058772 -0.30031 0.11332"
             rpy="1.5708 0.20867 -3.1416" />
         <parent link="chassis_link" />
-        <child link="rear_left_wheel_link" />
+        <child link="rear_right_wheel_link" />
         <axis xyz="0 0 -1" />
     </joint>
-    <!-- REAR RIGHT WHEEL -->
-    <link name="rear_right_wheel_link">
+    <!-- FRONT RIGHT WHEEL -->
+    <link name="front_right_wheel_link">
         <inertial>
             <origin
@@ -153,10 +153,10 @@
         </collision>
     </link>
-    <joint name="rear_right_wheel_joint" type="continuous">
+    <joint name="front_right_wheel_joint" type="continuous">
         <origin
             xyz="0.2863 -0.30031 0.11332"
             rpy="1.5708 0.19754 -3.1416" />
         <parent link="chassis_link" />
-        <child link="rear_right_wheel_link" />
+        <child link="front_right_wheel_link" />
         <axis xyz="0 0 -1" />
     </joint>

Commit message: wheels renamed and rviz rendering properly

File: rover_ros2/rover_description/urdf/wheels.xacro (robot description, xacro)
@@ -19,5 +19,5 @@
             <origin xyz="0 0 0" rpy="0 0 0" />
             <geometry>
-                <mesh filename="package://rover_description/meshes/front_left_wheel.STL" />
+                <mesh filename="package://rover_description/meshes/Wheel1.STL" />
             </geometry>
             <material name="">
@@ -29,5 +29,5 @@
             <origin xyz="0 0 0" rpy="0 0 0" />
             <geometry>
-                <mesh filename="package://rover_description/meshes/front_left_wheel.STL" />
+                <mesh filename="package://rover_description/meshes/Wheel1.STL" />
             </geometry>
         </collision>
@@ -59,5 +59,5 @@
             <origin xyz="0 0 0" rpy="0 0 0" />
             <geometry>
-                <mesh filename="package://rover_description/meshes/front_right_wheel.STL" />
+                <mesh filename="package://rover_description/meshes/Wheel2.STL" />
             </geometry>
             <material name="">
@@ -69,5 +69,5 @@
             <origin xyz="0 0 0" rpy="0 0 0" />
             <geometry>
-                <mesh filename="package://rover_description/meshes/front_right_wheel.STL" />
+                <mesh filename="package://rover_description/meshes/Wheel2.STL" />
             </geometry>
         </collision>
@@ -99,5 +99,5 @@
             <origin xyz="0 0 0" rpy="0 0 0" />
             <geometry>
-                <mesh filename="package://rover_description/meshes/rear_left_wheel.STL" />
+                <mesh filename="package://rover_description/meshes/Wheel3.STL" />
             </geometry>
             <material name="">
@@ -109,5 +109,5 @@
             <origin xyz="0 0 0" rpy="0 0 0" />
             <geometry>
-                <mesh filename="package://rover_description/meshes/rear_left_wheel.STL" />
+                <mesh filename="package://rover_description/meshes/Wheel3.STL" />
             </geometry>
         </collision>
@@ -139,5 +139,5 @@
             <origin xyz="0 0 0" rpy="0 0 0" />
             <geometry>
-                <mesh filename="package://rover_description/meshes/rear_right_wheel.STL" />
+                <mesh filename="package://rover_description/meshes/Wheel4.STL" />
             </geometry>
             <material name="">
@@ -149,5 +149,5 @@
             <origin xyz="0 0 0" rpy="0 0 0" />
             <geometry>
-                <mesh filename="package://rover_description/meshes/rear_right_wheel.STL" />
+                <mesh filename="package://rover_description/meshes/Wheel4.STL" />
             </geometry>
         </collision>

Commit message: fixed wheel axis misalignment causing driving drift

File: rover_ros2/rover_description/urdf/wheels.xacro (robot description, xacro)
@@ -36,5 +36,5 @@
         <origin
             xyz="0.2863 0 0.11332"
-            rpy="1.5708 -0.036526 0" />
+            rpy="0 ${pi/2} -${pi/2}" />
         <parent link="chassis_link" />
         <child link="front_left_wheel_link" />
@@ -76,5 +76,5 @@
         <origin
             xyz="-0.0058772 0 0.11332"
-            rpy="1.5708 -0.51093 0" />
+            rpy="0 ${pi/2} -${pi/2}" />
         <parent link="chassis_link" />
         <child link="rear_left_wheel_link" />
@@ -116,10 +116,9 @@
         <origin
             xyz="-0.0058772 -0.30031 0.11332"
-            rpy="1.5708 0.20867 -3.1416" />
+            rpy="-${pi/2} -${pi/2} 0" />
         <parent link="chassis_link" />
         <child link="rear_right_wheel_link" />
-        <axis xyz="0 0 -1" />
+        <axis xyz="0 0 1" />
     </joint>
-    <!-- TODO: This wheel is dragging a lot and causing the robot to turn while driving straight -->
     <!-- FRONT RIGHT WHEEL -->
     <link name="front_right_wheel_link">
@@ -157,8 +156,8 @@
         <origin
             xyz="0.2863 -0.30031 0.11332"
-            rpy="1.5708 0.19754 -3.1416" />
+            rpy="-${pi/2} -${pi/2} 0" />
         <parent link="chassis_link" />
         <child link="front_right_wheel_link" />
-        <axis xyz="0 0 -1" />
+        <axis xyz="0 0 1" />
     </joint>
 </robot>

Commit message: fixed wheel turning issue with left_wheel_reverse: true and added friction

File: rover_ros2/rover_description/urdf/wheels.xacro (robot description, xacro)
@@ -40,4 +40,6 @@
         <child link="front_left_wheel_link" />
         <axis xyz="0 0 -1" />
+        <limit effort="100" velocity="100"/>
+        <dynamics damping="0.0" friction="0.5"/>
     </joint>
     <!-- REAR LEFT WHEEL -->
@@ -80,4 +82,6 @@
         <child link="rear_left_wheel_link" />
         <axis xyz="0 0 -1" />
+        <limit effort="100" velocity="100"/>
+        <dynamics damping="0.0" friction="0.5"/>
     </joint>
     <!-- REAR RIGHT WHEEL -->
@@ -120,4 +124,6 @@
         <child link="rear_right_wheel_link" />
         <axis xyz="0 0 1" />
+        <limit effort="100" velocity="100"/>
+        <dynamics damping="0.0" friction="0.5"/>
     </joint>
     <!-- FRONT RIGHT WHEEL -->
@@ -160,4 +166,6 @@
         <child link="front_right_wheel_link" />
         <axis xyz="0 0 1" />
+        <limit effort="100" velocity="100"/>
+        <dynamics damping="0.0" friction="0.5"/>
     </joint>
 </robot>
