Commit message: added refined gazebo ros2 control and pure ros2 control conditionals

File: rover_ros2/rover_description/urdf/gazebo.xacro (robot description, xacro)
@@ -88,4 +88,41 @@
     <!-- ROS2 Control Plugin -->
     <xacro:if value="$(arg use_ros2_control)">
+        <ros2_control name="DiffDriveSystem" type="system">
+            <hardware>
+                <plugin>gz_ros2_control/GazeboSimSystem</plugin>
+            </hardware>
+            <joint name="front_left_wheel_joint">
+                <command_interface name="velocity">
+                    <param name="min">-10</param>
+                    <param name="max">10</param>
+                </command_interface>
+                <state_interface name="position"/>
+                <state_interface name="velocity"/>
+            </joint>
+            <joint name="rear_left_wheel_joint">
+                <command_interface name="velocity">
+                    <param name="min">-10</param>
+                    <param name="max">10</param>
+                </command_interface>
+                <state_interface name="position"/>
+                <state_interface name="velocity"/>
+            </joint>
+            <joint name="front_right_wheel_joint">
+                <command_interface name="velocity">
+                    <param name="min">-10</param>
+                    <param name="max">10</param>
+                </command_interface>
+                <state_interface name="position"/>
+                <state_interface name="velocity"/>
+            </joint>
+            <joint name="rear_right_wheel_joint">
+                <command_interface name="velocity">
+                    <param name="min">-10</param>
+                    <param name="max">10</param>
+                </command_interface>
+                <state_interface name="position"/>
+                <state_interface name="velocity"/>
+            </joint>
+        </ros2_control>
         <gazebo>
             <plugin filename="libgz_ros2_control-system.so" name="gz_ros2_control::GazeboSimROS2ControlPlugin">

Commit message: tried to fix weird turning and failed

File: rover_ros2/rover_description/urdf/gazebo.xacro (robot description, xacro)
@@ -8,4 +8,6 @@
     <gazebo reference="front_left_wheel_link">
         <material>Gazebo/Gray</material>
+        <mu1>0.55</mu1>
+        <mu2>0.4</mu2>
     </gazebo>
     <transmission name="front_left_wheel_transmission">
@@ -21,4 +23,6 @@
     <gazebo reference="front_right_wheel_link">
         <material>Gazebo/Gray</material>
+        <mu1>0.55</mu1>
+        <mu2>0.4</mu2>
     </gazebo>
     <transmission name="front_right_wheel_transmission">
@@ -34,4 +38,6 @@
     <gazebo reference="rear_left_wheel_link">
         <material>Gazebo/Gray</material>
+        <mu1>0.55</mu1>
+        <mu2>0.4</mu2>
     </gazebo>
     <transmission name="rear_left_wheel_transmission">
@@ -47,4 +53,6 @@
     <gazebo reference="rear_right_wheel_link">
         <material>Gazebo/Gray</material>
+        <mu1>0.55</mu1>
+        <mu2>0.4</mu2>
     </gazebo>
     <transmission name="rear_right_wheel_transmission">

File: rover_ros2/rover_description/urdf/wheels.xacro (robot description, xacro)
@@ -36,10 +36,9 @@
         <origin
             xyz="0.2863 0 0.11332"
-            rpy="0 ${pi/2} -${pi/2}" />
+            rpy="${pi/2} 0 0" />
         <parent link="chassis_link" />
         <child link="front_left_wheel_link" />
         <axis xyz="0 0 -1" />
         <limit effort="100" velocity="100"/>
-        <dynamics damping="0.0" friction="0.5"/>
     </joint>
     <!-- REAR LEFT WHEEL -->
@@ -78,10 +77,9 @@
         <origin
             xyz="-0.0058772 0 0.11332"
-            rpy="0 ${pi/2} -${pi/2}" />
+            rpy="${pi/2} 0 0" />
         <parent link="chassis_link" />
         <child link="rear_left_wheel_link" />
         <axis xyz="0 0 -1" />
         <limit effort="100" velocity="100"/>
-        <dynamics damping="0.0" friction="0.5"/>
     </joint>
     <!-- REAR RIGHT WHEEL -->
@@ -120,10 +118,9 @@
         <origin
             xyz="-0.0058772 -0.30031 0.11332"
-            rpy="-${pi/2} -${pi/2} 0" />
+            rpy="-${pi/2} 0 0" />
         <parent link="chassis_link" />
         <child link="rear_right_wheel_link" />
         <axis xyz="0 0 1" />
         <limit effort="100" velocity="100"/>
-        <dynamics damping="0.0" friction="0.5"/>
     </joint>
     <!-- FRONT RIGHT WHEEL -->
@@ -162,10 +159,9 @@
         <origin
             xyz="0.2863 -0.30031 0.11332"
-            rpy="-${pi/2} -${pi/2} 0" />
+            rpy="-${pi/2} 0 0" />
         <parent link="chassis_link" />
         <child link="front_right_wheel_link" />
         <axis xyz="0 0 1" />
         <limit effort="100" velocity="100"/>
-        <dynamics damping="0.0" friction="0.5"/>
     </joint>
 </robot>
